File: hardware/Sparrow-II/Interfaces&IO.kicad_sch (KiCad schematic)
At the start: 20 parts

Commit message: hardware: fixes connected to ERC errors 1/2
Parts:
- J_CAM1: footprint FC Drone Footprint Library:JST_BM03B-SRSS-TB_LF__SN_ -> SparrowHawk:JST_BM03B-SRSS-TB_LF__SN_
- J_ESC1: footprint FC Drone Footprint Library:JST_BM08B-SRSS-TB_LF__SN_ -> SparrowHawk:JST_BM08B-SRSS-TB_LF__SN_
- J_GPS1: footprint FC Drone Footprint Library:JST_BM06B-SRSS-TB_LF__SN_ -> SparrowHawk:JST_BM06B-SRSS-TB_LF__SN_
- J_RX1, J_VTX1: footprint FC Drone Footprint Library:JST_BM04B-SRSS-TB_LF__SN_ -> SparrowHawk:JST_BM04B-SRSS-TB_LF__SN_
Changed lines of the file:
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@@
 			)
 		)
-		(property "Footprint" "FC Drone Footprint Library:JST_BM06B-SRSS-TB_LF__SN_"
+		(property "Footprint" "SparrowHawk:JST_BM06B-SRSS-TB_LF__SN_"
 			(at 344.17 153.67 0)
 			(hide yes)
@@
 			)
 		)
-		(property "Footprint" "FC Drone Footprint Library:JST_BM04B-SRSS-TB_LF__SN_"
+		(property "Footprint" "SparrowHawk:JST_BM04B-SRSS-TB_LF__SN_"
 			(at 265.43 153.67 0)
 			(hide yes)
@@
 			)
 		)
-		(property "Footprint" "FC Drone Footprint Library:JST_BM08B-SRSS-TB_LF__SN_"
+		(property "Footprint" "SparrowHawk:JST_BM08B-SRSS-TB_LF__SN_"
 			(at 347.98 100.33 0)
 			(hide yes)
@@
 			)
 		)
-		(property "Footprint" "FC Drone Footprint Library:JST_BM04B-SRSS-TB_LF__SN_"
+		(property "Footprint" "SparrowHawk:JST_BM04B-SRSS-TB_LF__SN_"
 			(at 345.44 54.61 0)
 			(hide yes)
@@
 			)
 		)
-		(property "Footprint" "FC Drone Footprint Library:JST_BM03B-SRSS-TB_LF__SN_"
+		(property "Footprint" "SparrowHawk:JST_BM03B-SRSS-TB_LF__SN_"
 			(at 262.89 53.34 0)
 			(hide yes)
