File: hardware/Sparrow-II/Interfaces&IO.kicad_sch (KiCad schematic)
At the start: 20 parts

Commit message: hardware: BOM actualization and second layout
Parts:
- C_CURR_F1: footprint Capacitor_SMD:C_0402_1005Metric_Pad0.74x0.62mm_HandSolder -> Capacitor_SMD:C_0402_1005Metric; Dielectric (none) -> X7R; Voltage (none) -> 16V
- C_USB_SH1: footprint Capacitor_SMD:C_0402_1005Metric_Pad0.74x0.62mm_HandSolder -> Capacitor_SMD:C_0402_1005Metric; Note (none) -> Wylaczony: ekran USB zwarty do GND przez R_USB_SH1 = 0R; now not fitted; now left out of the parts list
- D_USB_VBUS1: MPN (none) -> PMEG2010AEH,115; Manufacturer (none) -> Nexperia
- J_CAM1: value BM03B-SRSS-TB_LF__SN_ -> CAM Pads; footprint SparrowHawk:JST_BM03B-SRSS-TB_LF__SN_ -> SparrowHawk:SolderPads_CAM_1x03; Availability In Stock -> (none); Check_prices https://www.snapeda.com/parts/BM03B-SRSS-TB(LF)(SN)/JST/vie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 -> (none); Description_1 Connector Header Surface Mount 3 position 0.039 (1.00mm) -> (none); MANUFACTURER JST Sales America Inc. -> (none); MAXIMUM_PACKAGE_HEIGHT 6.3 mm -> (none); MF JST Sales -> (none); MP BM03B-SRSS-TB(LF)(SN) -> (none); MPN (none) -> BM03B-SRSS-TB(LF)(SN); Manufacturer (none) -> JST Sales; Note (none) -> Pady lutownicze zamiast zlacza: 5V / GND / VIDEO_IN + 2 pad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; PARTREV N/A -> (none); Price None -> (none); Purchase-URL https://www.snapeda.com/api/url_track_click_mouser/?unipart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 -> (none); SNAPEDA_PN BM03B-SRSS-TB(LF)(SN) -> (none); STANDARD Manufacturer Recommendations -> (none); SnapEDA_Link https://www.snapeda.com/parts/BM03B-SRSS-TB(LF)(SN)/JST/vie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 -> (none); now left out of the parts list
- J_ESC1: Availability In Stock -> (none); Check_prices https://www.snapeda.com/parts/BM08B-SRSS-TB(LF)(SN)/JST/vie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 -> (none); Description_1 Connector Header Surface Mount 8 position 0.039 (1.00mm) -> (none); MANUFACTURER JST Sales America Inc. -> (none); MAXIMUM_PACKAGE_HEIGHT 6.3 mm -> (none); MF JST Sales -> (none); MP BM08B-SRSS-TB(LF)(SN) -> (none); MPN (none) -> BM08B-SRSS-TB(LF)(SN); Manufacturer (none) -> JST Sales; Note (none) -> PINOUT DO USTALENIA po wyborze 4in1 ESC - przepisac 1:1 z i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; PARTREV N/A -> (none); Price None -> (none); SNAPEDA_PN BM08B-SRSS-TB(LF)(SN) -> (none); STANDARD Manufacturer Recommendations -> (none); SnapEDA_Link https://www.snapeda.com/parts/BM08B-SRSS-TB(LF)(SN)/JST/vie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 -> (none)
- J_GPS1: Availability In Stock -> (none); Check_prices https://www.snapeda.com/parts/BM06B-SRSS-TB%20(LF)(SN)/JST/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 -> (none); Description_1 Connector Header Surface Mount 6 position 0.039 (1.00mm) -> (none); MANUFACTURER JST Sales America Inc. -> (none); MAXIMUM_PACKAGE_HEIGHT 6.3 mm -> (none); MF JST Sales -> (none); MP BM06B-SRSS-TB (LF)(SN) -> (none); MPN (none) -> BM06B-SRSS-TB (LF)(SN); Manufacturer (none) -> JST Sales; PARTREV N/A -> (none); Price None -> (none); Purchase-URL https://www.snapeda.com/api/url_track_click_mouser/?unipart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 -> (none); SNAPEDA_PN BM06B-SRSS-TB(LF)(SN) -> (none); STANDARD Manufacturer Recommendations -> (none); SnapEDA_Link https://www.snapeda.com/parts/BM06B-SRSS-TB%20(LF)(SN)/JST/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 -> (none)
- J_RX1: value BM04B-SRSS-TB_LF__SN_ -> RX Pads; footprint SparrowHawk:JST_BM04B-SRSS-TB_LF__SN_ -> SparrowHawk:SolderPads_RX_1x04; Availability In Stock -> (none); Check_prices https://www.snapeda.com/parts/BM04B-SRSS-TB(LF)(SN)/JST/vie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 -> (none); Description_1 Connector Header Surface Mount 4 position 0.039 (1.00mm) -> (none); MANUFACTURER JST Sales America Inc. -> (none); MAXIMUM_PACKAGE_HEIGHT 6.3 mm -> (none); MF JST Sales -> (none); MP BM04B-SRSS-TB(LF)(SN) -> (none); MPN (none) -> BM04B-SRSS-TB(LF)(SN); Manufacturer (none) -> JST Sales; Note (none) -> Pady lutownicze zamiast zlacza: 5V / GND / RX / TX + 2 pady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; PARTREV N/A -> (none); Price None -> (none); SNAPEDA_PN BM04B-SRSS-TB(LF)(SN) -> (none); STANDARD Manufacturer Recommendations -> (none); SnapEDA_Link https://www.snapeda.com/parts/BM04B-SRSS-TB(LF)(SN)/JST/vie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 -> (none); now left out of the parts list
- J_USB1: MPN (none) -> USB4085-GF-A; Manufacturer (none) -> GCT
- J_VTX1: value BM04B-SRSS-TB_LF__SN_ -> VTX Pads; footprint SparrowHawk:JST_BM04B-SRSS-TB_LF__SN_ -> SparrowHawk:SolderPads_VTX_1x04; Availability In Stock -> (none); Check_prices https://www.snapeda.com/parts/BM04B-SRSS-TB(LF)(SN)/JST/vie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 -> (none); Description_1 Connector Header Surface Mount 4 position 0.039 (1.00mm) -> (none); MANUFACTURER JST Sales America Inc. -> (none); MAXIMUM_PACKAGE_HEIGHT 6.3 mm -> (none); MF JST Sales -> (none); MP BM04B-SRSS-TB(LF)(SN) -> (none); MPN (none) -> BM04B-SRSS-TB(LF)(SN); Manufacturer (none) -> JST Sales; Note (none) -> Pad BAT = surowe VBAT. Na 6S to 25,2 V - sprawdz zakres wej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; PARTREV N/A -> (none); Price None -> (none); SNAPEDA_PN BM04B-SRSS-TB(LF)(SN) -> (none); STANDARD Manufacturer Recommendations -> (none); SnapEDA_Link https://www.snapeda.com/parts/BM04B-SRSS-TB(LF)(SN)/JST/vie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 -> (none); now left out of the parts list
- R_BZ_G1, R_BZ_PD1, R_CC1, R_CC2, R_CURR_F1: footprint Resistor_SMD:R_0402_1005Metric_Pad0.72x0.64mm_HandSolder -> Resistor_SMD:R_0402_1005Metric; Power (none) -> 0.063W; Tolerance (none) -> 1%
- R_USB_SH1: value 1M -> 0R; footprint Resistor_SMD:R_0402_1005Metric_Pad0.72x0.64mm_HandSolder -> Resistor_SMD:R_0402_1005Metric; Note (none) -> ekran USB-C wprost do GND (plytka ma jedna mase). Wczesniej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; Power (none) -> 0.063W; Tolerance (none) -> 1%
- U_ESD1: MPN (none) -> USBLC6-2SC6; Manufacturer (none) -> STMicroelectronics

Commit message: hardware: Layout improvement
Parts:
- BZ1, D_BZ1, J_BUZZER1, Q_BZ1, R_BZ_G1, R_BZ_PD1: now not fitted
Changed lines of the file:
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@@
 		(on_board no)
 		(in_pos_files yes)
-		(dnp no)
+		(dnp yes)
 		(fields_autoplaced yes)
 		(property "Reference" "R_BZ_G1"
@@
 			)
 		)
-		(property "Description" "Resistor"
+		(property "Description" "WYŁĄCZONY — rezystor bramkowy tranzystora buzzera"
 			(at 82.55 166.37 0)
 			(hide yes)
@@
 			)
 		)
-		(property "Description" "Resistor"
+		(property "Description" "Rezystor CC2 5,1 kΩ"
 			(at 113.03 91.44 0)
 			(hide yes)
@@
 		(on_board no)
 		(in_pos_files yes)
-		(dnp no)
+		(dnp yes)
 		(fields_autoplaced yes)
 		(property "Reference" "#PWR071"
@@
 		(on_board no)
 		(in_pos_files yes)
-		(dnp no)
+		(dnp yes)
 		(fields_autoplaced yes)
 		(property "Reference" "Q_BZ1"
@@
 			)
 		)
-		(property "Description" "30V Vds, 5.7A Id, N-Channel MOSFET, SOT-23"
+		(property "Description" "WYŁĄCZONY — tranzystor sterujący buzzerem. Obowiązkowy: PC13 ma limit 3 mA i nie może zasilać obciążenia"
 			(at 97.79 166.37 0)
 			(hide yes)
@@
 			)
 		)
-		(property "Datasheet" ""
+		(property "Datasheet" "https://www.jst-mfg.com/product/pdf/eng/eSH.pdf"
 			(at 344.17 153.67 0)
 			(hide yes)
@@
 			)
 		)
-		(property "Description" ""
+		(property "Description" "Złącze modułu GPS z kompasem: +5 V, UART2 i magistrala I2C"
 			(at 344.17 153.67 0)
 			(hide yes)
@@
 			)
 		)
-		(property "Description" "Unpolarized capacitor"
+		(property "Description" "WYŁĄCZONY (exclude BOM+board) — ekran idzie wprost do masy przez R_USB_SH1 = 0 Ω"
 			(at 57.15 99.06 0)
 			(hide yes)
@@
 			)
 		)
-		(property "Description" "20V, 1A very low Vf MEGA Schottky barrier rectifier, SOD-123F"
+		(property "Description" "Dioda ORująca zasilanie z USB do szyny +5 V. Pozwala skonfigurować płytkę bez pakietu i blokuje wsteczne zasilanie portu"
 			(at 153.67 63.5 0)
 			(hide yes)
@@
 		(on_board no)
 		(in_pos_files yes)
-		(dnp no)
+		(dnp yes)
 		(fields_autoplaced yes)
 		(property "Reference" "#PWR069"
@@
 		(on_board no)
 		(in_pos_files yes)
-		(dnp no)
+		(dnp yes)
 		(fields_autoplaced yes)
 		(property "Reference" "#PWR070"
@@
 		(on_board no)
 		(in_pos_files yes)
-		(dnp no)
+		(dnp yes)
 		(fields_autoplaced yes)
 		(property "Reference" "D_BZ1"
@@
 			)
 		)
-		(property "Description" "75V 0.15A Fast Switching Diode, SOD-123"
+		(property "Description" "WYŁĄCZONY — dioda gasząca dla buzzera"
 			(at 91.44 157.48 0)
 			(hide yes)
@@
 			)
 		)
-		(property "Description" ""
+		(property "Description" "Pady odbiornika RC (ELRS/CRSF/SBUS): 5 V, masa, UART1"
 			(at 265.43 153.67 0)
 			(hide yes)
@@
 			)
 		)
-		(property "Datasheet" ""
+		(property "Datasheet" "https://www.jst-mfg.com/product/pdf/eng/eSH.pdf"
 			(at 347.98 100.33 0)
 			(hide yes)
@@
 			)
 		)
-		(property "Description" ""
+		(property "Description" "Złącze taśmy do regulatora 4w1: zasilanie VBAT, sygnały M1–M4, pomiar prądu i telemetria. PINOUT DO USTALENIA po wyborze ESC"
 			(at 347.98 100.33 0)
 			(hide yes)
@@
 		(on_board no)
 		(in_pos_files yes)
-		(dnp no)
+		(dnp yes)
 		(fields_autoplaced yes)
 		(property "Reference" "R_BZ_PD1"
@@
 			)
 		)
-		(property "Description" "Resistor"
+		(property "Description" "WYŁĄCZONY — rezystor ściągający bramkę tranzystora buzzera"
 			(at 87.63 176.53 0)
 			(hide yes)
@@
 			)
 		)
-		(property "Description" "Resistor"
+		(property "Description" "Rezystor CC1 5,1 kΩ — deklaruje urządzenie jako odbiornik (sink) wg USB-C"
 			(at 124.46 91.44 0)
 			(hide yes)
@@
 			)
 		)
-		(property "Description" "Unpolarized capacitor"
+		(property "Description" "Kondensator filtru sygnału pomiaru prądu, stała czasowa 1 ms"
 			(at 261.62 97.79 0)
 			(hide yes)
@@
 			)
 		)
-		(property "Description" "Resistor"
+		(property "Description" "Zwarcie ekranu gniazda USB-C do masy. Płytka ma jedną masę, więc izolacja RC nie ma czego separować"
 			(at 76.2 99.06 0)
 			(hide yes)
@@
 			)
 		)
-		(property "Description" ""
+		(property "Description" "Pady nadajnika wideo: VBAT, sygnał wideo, UART sterowania. UWAGA: pad BAT to surowe 25,2 V na 6S"
 			(at 345.44 54.61 0)
 			(hide yes)
@@
 			)
 		)
-		(property "Description" "USB 2.0-only 16P Type-C Receptacle connector"
+		(property "Description" "Gniazdo USB-C. Konfiguracja i aktualizacja firmware; 16 pinów daje wytrzymałość mechaniczną często wtykanego portu"
 			(at 83.82 71.12 0)
 			(hide yes)
@@
 			)
 		)
-		(property "Description" "Resistor"
+		(property "Description" "Rezystor filtru sygnału pomiaru prądu z ESC. Ogranicza też prąd wstrzykiwany, gdyby regulator podał 5 V"
 			(at 275.59 93.98 0)
 			(hide yes)
@@
 			)
 		)
-		(property "Description" "Very low capacitance ESD protection diode, 2 data-line, SOT-23-6"
+		(property "Description" "Ochrona ESD linii danych USB. Wpięty przelotowo w D+/D−"
 			(at 153.67 88.9 0)
 			(hide yes)
@@
 		(on_board no)
 		(in_pos_files yes)
-		(dnp no)
+		(dnp yes)
 		(fields_autoplaced yes)
 		(property "Reference" "BZ1"
@@
 			)
 		)
-		(property "Description" "Buzzer, polarized"
+		(property "Description" "WYŁĄCZONY (exclude BOM+board) — buzzer sygnalizacyjny"
 			(at 120.65 143.51 0)
 			(hide yes)
@@
 			)
 		)
-		(property "Description" ""
+		(property "Description" "Pady kamery analogowej: 5 V filtrowane, masa, sygnał wideo"
 			(at 262.89 53.34 0)
 			(hide yes)
@@
 		(on_board no)
 		(in_pos_files yes)
-		(dnp no)
+		(dnp yes)
 		(fields_autoplaced yes)
 		(property "Reference" "J_BUZZER1"
@@
 			)
 		)
-		(property "Description" "Generic connector, single row, 01x02, script generated (kicad-library-utils/schlib/autogen/connector/)"
+		(property "Description" "WYŁĄCZONY — złącze buzzera zewnętrznego"
 			(at 123.19 153.67 0)
 			(hide yes)

Commit message: hardware: layout checkpoint 3 - fixed DRC
Connections:
- net USB_C_DM renamed USB_C_DN
- net USB_DM renamed USB_DN
Changed lines of the file:
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@@
 		)
 	)
-	(label "USB_C_DM"
+	(label "USB_C_DN"
 		(at 101.6 71.12 0)
 		(effects
@@
 		)
 	)
-	(label "USB_C_DM"
+	(label "USB_C_DN"
 		(at 146.05 91.44 180)
 		(effects
@@
 		)
 	)
-	(hierarchical_label "USB_DM"
+	(hierarchical_label "USB_DN"
 		(shape bidirectional)
 		(at 161.29 91.44 0)
