File: hardware/Sparrow-II/Video&OSD.kicad_sch (KiCad schematic)
At the start: 16 parts

Commit message: hardware: fixes connected to ERC errors 1/2
Parts:
- U_OSD1: footprint FC Drone Footprint Library:SOP65P640X120-29N -> SparrowHawk:SOP65P640X120-29N
Changed lines of the file:
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@@
 			)
 		)
-		(property "Footprint" "FC Drone Footprint Library:SOP65P640X120-29N"
+		(property "Footprint" "SparrowHawk:SOP65P640X120-29N"
 			(at 214.63 166.04 0)
 			(hide yes)
