File: hardware/Sparrow-II/Video&OSD.kicad_sch (KiCad schematic)
At the start: 16 parts

Commit message: hardware: OSD quick fixes
Parts:
- added R_VID_BYPASS1: 0R, Resistor_SMD:R_0402_1005Metric_Pad0.72x0.64mm_HandSolder, symbol Device:R
Connections:
- net GND: no longer U_OSD1.3 (DVDD)
- net VIDEO_IN: now also R_VID_BYPASS1.1
- net VIDEO_OUT: now also R_VID_BYPASS1.2
- net +5V renamed +3V3
- net +3V3: now also U_OSD1.3 (DVDD)
- net +5_VIDEO renamed +5V_VIDEO
Other:
- note added: "OBEJSCIE OSD - AWARYJNE"
Changed lines of the file:
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@@
 	(rectangle
 		(start 133.604 21.336)
-		(end 326.644 157.48)
+		(end 326.644 177.546)
 		(stroke
 			(width 0)
@@
 		)
 	)
+	(text "OBEJSCIE OSD - AWARYJNE"
+		(exclude_from_sim no)
+		(at 279.654 148.844 0)
+		(effects
+			(font
+				(size 1.27 1.27)
+			)
+			(justify left bottom)
+		)
+	)
 	(junction
-		(at 163.83 71.12)
+		(at 163.83 63.5)
 		(diameter 0)
 		(color 0 0 0 0)
@@
 	(wire
 		(pts
+			(xy 163.83 63.5) (xy 166.37 63.5)
+		)
+		(stroke
+			(width 0)
+			(type default)
+		)
+	)
+	(wire
+		(pts
 			(xy 44.45 66.04) (xy 49.53 66.04)
 		)
@@
 	(wire
 		(pts
+			(xy 295.91 160.02) (xy 302.26 160.02)
+		)
+		(stroke
+			(width 0)
+			(type default)
+		)
+	)
+	(wire
+		(pts
 			(xy 57.15 53.34) (xy 66.04 53.34)
 		)
@@
 	(wire
 		(pts
+			(xy 166.37 76.2) (xy 166.37 63.5)
+		)
+		(stroke
+			(width 0)
+			(type default)
+		)
+	)
+	(wire
+		(pts
 			(xy 227.33 132.08) (xy 231.14 132.08)
 		)
@@
 	(wire
 		(pts
+			(xy 288.29 160.02) (xy 281.94 160.02)
+		)
+		(stroke
+			(width 0)
+			(type default)
+		)
+	)
+	(wire
+		(pts
 			(xy 71.12 59.69) (xy 71.12 78.74)
 		)
@@
 	(wire
 		(pts
-			(xy 163.83 71.12) (xy 166.37 71.12)
-		)
-		(stroke
-			(width 0)
-			(type default)
-		)
-	)
-	(wire
-		(pts
 			(xy 284.48 105.41) (xy 284.48 106.68)
-		)
-		(stroke
-			(width 0)
-			(type default)
-		)
-	)
-	(wire
-		(pts
-			(xy 166.37 71.12) (xy 166.37 76.2)
 		)
 		(stroke
@@
 		)
 	)
+	(label "VIDEO_OUT"
+		(at 302.26 160.02 0)
+		(effects
+			(font
+				(size 1.27 1.27)
+			)
+			(justify left bottom)
+		)
+	)
+	(label "VIDEO_IN"
+		(at 281.94 160.02 180)
+		(effects
+			(font
+				(size 1.27 1.27)
+			)
+			(justify right bottom)
+		)
+	)
 	(label "OSD_CLK_OUT"
 		(at 175.26 83.82 180)
@@
 		)
 	)
-	(global_label "+5_VIDEO"
+	(global_label "+5V_VIDEO"
 		(shape input)
 		(at 248.92 102.87 90)
@@
 		)
 	)
-	(global_label "+5_VIDEO"
+	(global_label "+5V_VIDEO"
 		(shape input)
 		(at 273.05 64.77 90)
@@
 		)
 	)
-	(global_label "+5_VIDEO"
+	(global_label "+5V_VIDEO"
 		(shape input)
 		(at 308.61 86.36 90)
@@
 	)
 	(symbol
+		(lib_id "power:+3V3")
+		(at 231.14 118.11 0)
+		(unit 1)
+		(body_style 1)
+		(exclude_from_sim no)
+		(in_bom yes)
+		(on_board yes)
+		(in_pos_files yes)
+		(dnp no)
+		(fields_autoplaced yes)
+		(property "Reference" "#PWR086"
+			(at 231.14 121.92 0)
+			(hide yes)
+			(show_name no)
+			(do_not_autoplace no)
+			(effects
+				(font
+					(size 1.27 1.27)
+				)
+			)
+		)
+		(property "Value" "+3V3"
+			(at 231.14 113.03 0)
+			(show_name no)
+			(do_not_autoplace no)
+			(effects
+				(font
+					(size 1.27 1.27)
+				)
+			)
+		)
+		(property "Footprint" ""
+			(at 231.14 118.11 0)
+			(hide yes)
+			(show_name no)
+			(do_not_autoplace no)
+			(effects
+				(font
+					(size 1.27 1.27)
+				)
+			)
+		)
+		(property "Datasheet" ""
+			(at 231.14 118.11 0)
+			(hide yes)
+			(show_name no)
+			(do_not_autoplace no)
+			(effects
+				(font
+					(size 1.27 1.27)
+				)
+			)
+		)
+		(property "Description" "Power symbol creates a global label with name \"+5V\""
+			(at 231.14 118.11 0)
+			(hide yes)
+			(show_name no)
+			(do_not_autoplace no)
+			(effects
+				(font
+					(size 1.27 1.27)
+				)
+			)
+		)
+		(pin "1"
+		)
+		(instances
+			(project "Flight Controller"
+				(path "/64d08664-7c2b-4b48-a9dd-dae3f797396a/21e0c0df-5477-4a68-8911-aafd9a2904df"
+					(reference "#PWR086")
+					(unit 1)
+				)
+			)
+		)
+	)
+	(symbol
 		(lib_id "power:GND")
 		(at 200.66 127 0)
@@
 	)
 	(symbol
-		(lib_id "power:+5V")
+		(lib_id "power:+3V3")
 		(at 163.83 62.23 0)
 		(unit 1)
@@
 			)
 		)
-		(property "Value" "+5V"
+		(property "Value" "+3V3"
 			(at 163.83 57.15 0)
 			(show_name no)
@@
 	)
 	(symbol
-		(lib_id "power:+5V")
-		(at 231.14 118.11 0)
-		(unit 1)
-		(body_style 1)
-		(exclude_from_sim no)
-		(in_bom yes)
-		(on_board yes)
-		(in_pos_files yes)
-		(dnp no)
-		(fields_autoplaced yes)
-		(property "Reference" "#PWR056"
-			(at 231.14 121.92 0)
-			(hide yes)
-			(show_name no)
-			(do_not_autoplace no)
-			(effects
-				(font
-					(size 1.27 1.27)
-				)
-			)
-		)
-		(property "Value" "+5V"
-			(at 233.68 116.8399 0)
-			(show_name no)
-			(do_not_autoplace no)
-			(effects
-				(font
-					(size 1.27 1.27)
-				)
-				(justify left)
-			)
-		)
-		(property "Footprint" ""
-			(at 231.14 118.11 0)
-			(hide yes)
-			(show_name no)
-			(do_not_autoplace no)
-			(effects
-				(font
-					(size 1.27 1.27)
-				)
-			)
-		)
-		(property "Datasheet" ""
-			(at 231.14 118.11 0)
-			(hide yes)
-			(show_name no)
-			(do_not_autoplace no)
-			(effects
-				(font
-					(size 1.27 1.27)
-				)
-			)
-		)
-		(property "Description" "Power symbol creates a global label with name \"+5V\""
-			(at 231.14 118.11 0)
-			(hide yes)
-			(show_name no)
-			(do_not_autoplace no)
-			(effects
-				(font
-					(size 1.27 1.27)
-				)
-			)
-		)
-		(pin "1"
-		)
-		(instances
-			(project "Flight Controller"
-				(path "/64d08664-7c2b-4b48-a9dd-dae3f797396a/21e0c0df-5477-4a68-8911-aafd9a2904df"
-					(reference "#PWR056")
-					(unit 1)
-				)
-			)
-		)
-	)
-	(symbol
 		(lib_id "power:GND")
 		(at 233.68 91.44 0)
@@
 					(unit 1)
 				)
+			)
+		)
+	)
+	(symbol
+		(lib_id "Device:R")
+		(at 292.1 160.02 90)
+		(unit 1)
+		(body_style 1)
+		(exclude_from_sim no)
+		(in_bom yes)
+		(on_board yes)
+		(in_pos_files yes)
+		(dnp yes)
+		(fields_autoplaced yes)
+		(property "Reference" "R_VID_BYPASS1"
+			(at 292.1 157.48 0)
+			(show_name no)
+			(do_not_autoplace no)
+			(effects
+				(font
+					(size 1.27 1.27)
+				)
+			)
+		)
+		(property "Value" "0R"
+			(at 292.1 162.56 0)
+			(show_name no)
+			(do_not_autoplace no)
+			(effects
+				(font
+					(size 1.27 1.27)
+				)
+			)
+		)
+		(property "Footprint" "Resistor_SMD:R_0402_1005Metric_Pad0.72x0.64mm_HandSolder"
+			(at 292.1 160.02 0)
+			(hide yes)
+			(show_name no)
+			(do_not_autoplace no)
+			(effects
+				(font
+					(size 1.27 1.27)
+				)
+			)
+		)
+		(property "Datasheet" ""
+			(at 292.1 160.02 0)
+			(hide yes)
+			(show_name no)
+			(do_not_autoplace no)
+			(effects
+				(font
+					(size 1.27 1.27)
+				)
+			)
+		)
+		(property "Description" "Resistor"
+			(at 292.1 160.02 0)
+			(hide yes)
+			(show_name no)
+			(do_not_autoplace no)
+			(effects
+				(font
+					(size 1.27 1.27)
+				)
+			)
+		)
+		(pin "1"
+		)
+		(pin "2"
+		)
+		(instances
+			(project "Flight Controller"
+				(path "/64d08664-7c2b-4b48-a9dd-dae3f797396a/21e0c0df-5477-4a68-8911-aafd9a2904df"
+					(reference "R_VID_BYPASS1")
+					(unit 1)
+				)

Commit message: hardware: VDD pins fix; OSD floating pin
Connections:
- net GND: now also U_OSD1.13 (SYNC_IN)
- no-connect marks 12 -> 11
Changed lines of the file:
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@@
 	)
 	(no_connect
-		(at 182.88 101.6)
-	)
-	(no_connect
 		(at 182.88 86.36)
 	)
@@
 					(unit 1)
 				)
+			)
+		)
+	)
+	(wire
+		(pts
+			(xy 182.88 101.6) (xy 175.26 101.6)
+		)
+		(stroke
+			(width 0)
+			(type default)
+		)
+	)
+	(symbol
+		(lib_id "power:GND")
+		(at 175.26 101.6 0)
+		(unit 1)
+		(body_style 1)
+		(exclude_from_sim no)
+		(in_bom yes)
+		(on_board yes)
+		(in_pos_files yes)
+		(dnp no)
+		(fields_autoplaced yes)
+		(property "Reference" "#PWR090"
+			(at 175.26 98.425 0)
+			(hide yes)
+			(show_name no)
+			(do_not_autoplace no)
+			(effects
+				(font
+					(size 1.27 1.27)
+				)
+			)
+		)
+		(property "Value" "GND"
+			(at 175.26 104.77499999999999 0)
+			(show_name no)
+			(do_not_autoplace no)
+			(effects
+				(font
+					(size 1.27 1.27)
+				)
+			)
+		)
+		(property "Footprint" ""
+			(at 175.26 101.6 0)
+			(hide yes)
+			(show_name no)
+			(do_not_autoplace no)
+			(effects
+				(font
+					(size 1.27 1.27)
+				)
+			)
+		)
+		(property "Datasheet" ""
+			(at 175.26 101.6 0)
+			(hide yes)
+			(show_name no)
+			(do_not_autoplace no)
+			(effects
+				(font
+					(size 1.27 1.27)
+				)
+			)
+		)
+		(property "Description" "Power symbol"
+			(at 175.26 101.6 0)
+			(hide yes)
+			(show_name no)
+			(do_not_autoplace no)
+			(effects
+				(font
+					(size 1.27 1.27)
+				)
+			)
+		)
+		(pin "1"
+		)
+		(instances
+			(project "Flight Controller"
+				(path "/64d08664-7c2b-4b48-a9dd-dae3f797396a/21e0c0df-5477-4a68-8911-aafd9a2904df"
+					(reference "#PWR090")
+					(unit 1)
+				)

Commit message: hardware: change in oscilator values
Parts:
- R_HSE1: value 1k -> 0R
Changed lines of the file:
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@@
 	(wire
 		(pts
+			(xy 182.88 101.6) (xy 175.26 101.6)
+		)
+		(stroke
+			(width 0)
+			(type default)
+		)
+	)
+	(wire
+		(pts
 			(xy 218.44 81.28) (xy 236.22 81.28)
 		)
@@
 	(symbol
 		(lib_id "power:GND")
+		(at 175.26 101.6 0)
+		(unit 1)
+		(body_style 1)
+		(exclude_from_sim no)
+		(in_bom yes)
+		(on_board yes)
+		(in_pos_files yes)
+		(dnp no)
+		(fields_autoplaced yes)
+		(property "Reference" "#PWR090"
+			(at 175.26 98.425 0)
+			(hide yes)
+			(show_name no)
+			(do_not_autoplace no)
+			(effects
+				(font
+					(size 1.27 1.27)
+				)
+			)
+		)
+		(property "Value" "GND"
+			(at 175.26 104.775 0)
+			(show_name no)
+			(do_not_autoplace no)
+			(effects
+				(font
+					(size 1.27 1.27)
+				)
+			)
+		)
+		(property "Footprint" ""
+			(at 175.26 101.6 0)
+			(hide yes)
+			(show_name no)
+			(do_not_autoplace no)
+			(effects
+				(font
+					(size 1.27 1.27)
+				)
+			)
+		)
+		(property "Datasheet" ""
+			(at 175.26 101.6 0)
+			(hide yes)
+			(show_name no)
+			(do_not_autoplace no)
+			(effects
+				(font
+					(size 1.27 1.27)
+				)
+			)
+		)
+		(property "Description" "Power symbol"
+			(at 175.26 101.6 0)
+			(hide yes)
+			(show_name no)
+			(do_not_autoplace no)
+			(effects
+				(font
+					(size 1.27 1.27)
+				)
+			)
+		)
+		(pin "1"
+		)
+		(instances
+			(project "Flight Controller"
+				(path "/64d08664-7c2b-4b48-a9dd-dae3f797396a/21e0c0df-5477-4a68-8911-aafd9a2904df"
+					(reference "#PWR090")
+					(unit 1)
+				)
+			)
+		)
+	)
+	(symbol
+		(lib_id "power:GND")
 		(at 233.68 91.44 0)
 		(unit 1)
@@
 			)
 		)
-		(property "Value" "1k"
+		(property "Value" "0R"
 			(at 77.47 62.23 90)
 			(show_name no)
@@
 					(unit 1)
 				)
-			)
-		)
-	)
-	(wire
-		(pts
-			(xy 182.88 101.6) (xy 175.26 101.6)
-		)
-		(stroke
-			(width 0)
-			(type default)
-		)
-	)
-	(symbol
-		(lib_id "power:GND")
-		(at 175.26 101.6 0)
-		(unit 1)
-		(body_style 1)
-		(exclude_from_sim no)
-		(in_bom yes)
-		(on_board yes)
-		(in_pos_files yes)
-		(dnp no)
-		(fields_autoplaced yes)
-		(property "Reference" "#PWR090"
-			(at 175.26 98.425 0)
-			(hide yes)
-			(show_name no)
-			(do_not_autoplace no)
-			(effects
-				(font
-					(size 1.27 1.27)
-				)
-			)
-		)
-		(property "Value" "GND"
-			(at 175.26 104.77499999999999 0)
-			(show_name no)
-			(do_not_autoplace no)
-			(effects
-				(font
-					(size 1.27 1.27)
-				)
-			)
-		)
-		(property "Footprint" ""
-			(at 175.26 101.6 0)
-			(hide yes)
-			(show_name no)
-			(do_not_autoplace no)
-			(effects
-				(font
-					(size 1.27 1.27)
-				)
-			)
-		)
-		(property "Datasheet" ""
-			(at 175.26 101.6 0)
-			(hide yes)
-			(show_name no)
-			(do_not_autoplace no)
-			(effects
-				(font
-					(size 1.27 1.27)
-				)
-			)
-		)
-		(property "Description" "Power symbol"
-			(at 175.26 101.6 0)
-			(hide yes)
-			(show_name no)
-			(do_not_autoplace no)
-			(effects
-				(font
-					(size 1.27 1.27)
-				)
-			)
-		)
-		(pin "1"
-		)
-		(instances
-			(project "Flight Controller"
-				(path "/64d08664-7c2b-4b48-a9dd-dae3f797396a/21e0c0df-5477-4a68-8911-aafd9a2904df"
-					(reference "#PWR090")
-					(unit 1)
-				)

Commit message: hardware: BOM actualization and second layout
Parts:
- C_OSD_AVDD1, C_OSD_DVDD1, C_OSD_PVDD2, C_VID_IN_AC1: footprint Capacitor_SMD:C_0402_1005Metric_Pad0.74x0.62mm_HandSolder -> Capacitor_SMD:C_0402_1005Metric; Dielectric (none) -> X7R; Voltage (none) -> 16V
- C_OSD_PVDD1: footprint Capacitor_SMD:C_0402_1005Metric_Pad0.74x0.62mm_HandSolder -> Capacitor_SMD:C_0603_1608Metric; Dielectric (none) -> X7R; Voltage (none) -> 16V
- C_OSD_SAG1: footprint Capacitor_SMD:C_0402_1005Metric_Pad0.74x0.62mm_HandSolder -> Capacitor_SMD:C_0805_2012Metric; Dielectric (none) -> X5R; Note (none) -> CSAG wg AT7456E tab.2 (COUT 22uF + CSAG 22uF = 0.4% line-ti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; Voltage (none) -> 10V
- C_OSD_XTAL1, C_OSD_XTAL2: footprint Capacitor_SMD:C_0402_1005Metric_Pad0.74x0.62mm_HandSolder -> Capacitor_SMD:C_0402_1005Metric; Dielectric (none) -> C0G/NP0; Voltage (none) -> 50V
- C_VID_OUT_AC1: footprint Capacitor_SMD:C_0402_1005Metric_Pad0.74x0.62mm_HandSolder -> Capacitor_SMD:C_0805_2012Metric; Dielectric (none) -> X5R; Note (none) -> COUT wg AT7456E tab.2; Voltage (none) -> 10V
- D_VID_CLAMP1: MPN (none) -> BAV99,215; Manufacturer (none) -> Nexperia
- R_HSE1, R_OSD_RST1, R_VID_BYPASS1, R_VID_IN_T1, R_VID_OUT_T1: footprint Resistor_SMD:R_0402_1005Metric_Pad0.72x0.64mm_HandSolder -> Resistor_SMD:R_0402_1005Metric; Power (none) -> 0.063W; Tolerance (none) -> 1%
- U_OSD1: MPN (none) -> AT7456E; Manufacturer (none) -> ICOF; Manufacturer_Name ICOF -> (none); Manufacturer_Part_Number AT7456E -> (none)
- Y_OSD1: footprint Crystal:Crystal_SMD_3225-4Pin_3.2x2.5mm_HandSoldering -> Crystal:Crystal_SMD_3225-4Pin_3.2x2.5mm; MPN (none) -> ABM8-27.000MHZ-B2-T; Manufacturer (none) -> Abracon; Note (none) -> numer katalogowy do potwierdzenia u dystrybutora; Spec (none) -> 27MHz, CL=18pF, ESR 50R

Commit message: hardware: Layout improvement
Parts:
- Y_OSD1: Spec 27MHz, CL=18pF, ESR 50R -> 27 MHz, CL = 18 pF, ESR 50 Ω, obudowa 3225 4-pad
Changed lines of the file:
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@@
 			)
 		)
-		(property "Description" "Unpolarized capacitor"
+		(property "Description" "Odsprzęganie zasilania analogowego OSD"
 			(at 248.92 106.68 0)
 			(hide yes)
@@
 			)
 		)
-		(property "Description" "Resistor"
+		(property "Description" "Terminacja 75 Ω wejścia wideo z kamery"
 			(at 284.48 101.6 0)
 			(hide yes)
@@
 			)
 		)
-		(property "Description" "Unpolarized capacitor"
+		(property "Description" "Kondensator sprzęgający wyjścia wideo (COUT). Wartość powiązana z C_OSD_SAG1"
 			(at 231.14 58.42 0)
 			(hide yes)
@@
 			)
 		)
-		(property "Description" "Resistor"
+		(property "Description" "Rezystor szeregowy 75 Ω wyjścia wideo do nadajnika"
 			(at 251.46 48.26 0)
 			(hide yes)
@@
 			)
 		)
-		(property "Description" "Unpolarized capacitor"
+		(property "Description" "Sprzężenie zmiennoprądowe wejścia wideo z kamery — odcina składową stałą"
 			(at 284.48 90.17 0)
 			(hide yes)
@@
 			)
 		)
-		(property "Description" "Unpolarized capacitor"
+		(property "Description" "Zapas ładunku dla stopnia wyjściowego wideo"
 			(at 252.73 69.85 0)
 			(hide yes)
@@
 			)
 		)
-		(property "Description" "Unpolarized capacitor"
+		(property "Description" "Kondensator korekcji zwisu (CSAG). Para 22 µF + 22 µF z C_VID_OUT_AC1 daje 0,4 % zniekształcenia line-time wg Tabeli 2 datasheetu AT7456E"
 			(at 251.46 58.42 0)
 			(hide yes)
@@
 			)
 		)
-		(property "Datasheet" ""
+		(property "Datasheet" "https://abracon.com/Resonators/ABM8.pdf"
 			(at 66.04 59.69 0)
 			(hide yes)
@@
 			)
 		)
-		(property "Description" "Four pin crystal, GND on pins 2 and 4"
+		(property "Description" "Kwarc 27 MHz — zegar próbkowania toru wideo OSD"
 			(at 66.04 59.69 0)
 			(hide yes)
@@
 			)
 		)
-		(property "Spec" "27MHz, CL=18pF, ESR 50R"
+		(property "Spec" "27 MHz, CL = 18 pF, ESR 50 Ω, obudowa 3225 4-pad"
 			(at 66.04 59.69 0)
 			(hide yes)
@@
 			)
 		)
-		(property "Description" "Unpolarized capacitor"
+		(property "Description" "Odsprzęganie HF stopnia wyjściowego wideo"
 			(at 273.05 69.85 0)
 			(hide yes)
@@
 			)
 		)
-		(property "Description" "Unpolarized capacitor"
+		(property "Description" "Kondensator obciążenia kwarcu 27 MHz, C0G"
 			(at 53.34 53.34 0)
 			(hide yes)
@@
 			)
 		)
-		(property "Description" "Unpolarized capacitor"
+		(property "Description" "Drugi kondensator obciążenia kwarcu 27 MHz, C0G"
 			(at 53.34 66.04 0)
 			(hide yes)
@@
 			)
 		)
-		(property "Description" "Video Character Overlay Chip (OSD)"
+		(property "Description" "Generator napisów OSD, odpowiednik MAX7456. Nakłada telemetrię na analogowy sygnał wideo"
 			(at 182.88 71.12 0)
 			(hide yes)
@@
 			)
 		)
-		(property "Description" "BAV99 High-speed switching diodes, SOT-23"
+		(property "Description" "Ogranicznik sygnału wideo. Para szeregowa: pad 3 (VIDEO_IN) jest złączem, obcina poniżej −0,7 V i powyżej +5,7 V"
 			(at 308.61 93.98 0)
 			(hide yes)
@@
 			)
 		)
-		(property "Description" "Resistor"
+		(property "Description" "NIE MONTOWAĆ. Zworka ratunkowa omijająca OSD — do zamontowania tylko gdyby sekcja OSD nie zadziałała. Przy działającym OSD zwierałaby wyjście z wejściem"
 			(at 292.1 160.02 0)
 			(hide yes)
@@
 			)
 		)
-		(property "Description" "Resistor"
+		(property "Description" "Rezystor szeregowy oscylatora OSD, 0 Ω. Układ referencyjny MAX7456 nie ma tu rezystora — przy 1 kΩ kwarc by nie wystartował"
 			(at 77.47 66.04 0)
 			(hide yes)
@@
 			)
 		)
-		(property "Description" "Unpolarized capacitor"
+		(property "Description" "Odsprzęganie zasilania cyfrowego OSD. DVDD na +3V3, bo próg wejściowy to 0,65 × VDVDD"
 			(at 163.83 67.31 0)
 			(hide yes)
@@
 			)
 		)
-		(property "Description" "Resistor"
+		(property "Description" "Podciągnięcie linii /RESET OSD"
 			(at 231.14 125.73 0)
 			(hide yes)

Commit message: hardware: layout checkpoint 3 - fixed DRC
Parts:
- removed R_HSE1: 0R, Resistor_SMD:R_0402_1005Metric, symbol Device:R
Connections:
- net OSD_CLK_OUT: now also C_OSD_XTAL2.2, Y_OSD1.1
Changed lines of the file:
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@@
 	(wire
 		(pts
+			(xy 73.66 66.04) (xy 81.28 66.04)
+		)
+		(stroke
+			(width 0)
+			(type default)
+		)
+	)
+	(wire
+		(pts
 			(xy 233.68 62.23) (xy 251.46 62.23)
 		)
@@
 			)
 		)
-	)
-	(symbol
-		(lib_id "Device:R")
-		(at 77.47 66.04 90)
-		(unit 1)
-		(body_style 1)
-		(exclude_from_sim no)
-		(in_bom yes)
-		(on_board yes)
-		(in_pos_files yes)
-		(dnp no)
-		(fields_autoplaced yes)
-		(property "Reference" "R_HSE1"
-			(at 77.47 59.69 90)
-			(show_name no)
-			(do_not_autoplace no)
-			(effects
-				(font
-					(size 1.27 1.27)
-				)
-			)
-		)
-		(property "Value" "0R"
-			(at 77.47 62.23 90)
-			(show_name no)
-			(do_not_autoplace no)
-			(effects
-				(font
-					(size 1.27 1.27)
-				)
-			)
-		)
-		(property "Footprint" "Resistor_SMD:R_0402_1005Metric"
-			(at 77.47 67.818 90)
-			(hide yes)
-			(show_name no)
-			(do_not_autoplace no)
-			(effects
-				(font
-					(size 1.27 1.27)
-				)
-			)
-		)
-		(property "Datasheet" ""
-			(at 77.47 66.04 0)
-			(hide yes)
-			(show_name no)
-			(do_not_autoplace no)
-			(effects
-				(font
-					(size 1.27 1.27)
-				)
-			)
-		)
-		(property "Description" "Rezystor szeregowy oscylatora OSD, 0 Ω. Układ referencyjny MAX7456 nie ma tu rezystora — przy 1 kΩ kwarc by nie wystartował"
-			(at 77.47 66.04 0)
-			(hide yes)
-			(show_name no)
-			(do_not_autoplace no)
-			(effects
-				(font
-					(size 1.27 1.27)
-				)
-			)
-		)
-		(property "Tolerance" "1%"
-			(at 77.47 66.04 0)
-			(hide yes)
-			(show_name no)
-			(do_not_autoplace no)
-			(effects
-				(font
-					(size 1.27 1.27)
-				)
-			)
-		)
-		(property "Power" "0.063W"
-			(at 77.47 66.04 0)
-			(hide yes)
-			(show_name no)
-			(do_not_autoplace no)
-			(effects
-				(font
-					(size 1.27 1.27)
-				)
-			)
-		)
-		(pin "2"
-		)
-		(pin "1"
-		)
-		(instances
-			(project "Flight Controller"
-				(path "/64d08664-7c2b-4b48-a9dd-dae3f797396a/21e0c0df-5477-4a68-8911-aafd9a2904df"
-					(reference "R_HSE1")
-					(unit 1)
-				)
-			)
-		)
-	)
-	(symbol
+	)	(symbol
 		(lib_id "Device:C")
 		(at 163.83 67.31 180)

Commit message: hardware: decoupling capacitors route
Changed lines of the file:
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@@
 	(wire
 		(pts
-			(xy 73.66 66.04) (xy 81.28 66.04)
-		)
-		(stroke
-			(width 0)
-			(type default)
-		)
-	)
-	(wire
-		(pts
 			(xy 233.68 62.23) (xy 251.46 62.23)
 		)
@@
 	(wire
 		(pts
-			(xy 66.04 66.04) (xy 73.66 66.04)
+			(xy 66.04 66.04) (xy 85.09 66.04)
 		)
 		(stroke
@@
 	(wire
 		(pts
-			(xy 81.28 66.04) (xy 85.09 66.04)
-		)
-		(stroke
-			(width 0)
-			(type default)
-		)
-	)
-	(wire
-		(pts
 			(xy 252.73 73.66) (xy 273.05 73.66)
 		)
@@
 			)
 		)
-	)	(symbol
+	)
+	(symbol
 		(lib_id "Device:C")
 		(at 163.83 67.31 180)
