File: hardware/Sparrow-II/Flight Controller.kicad_sch (KiCad schematic)
At the start: 12 parts

Commit message: hardware: BOM actualization and second layout
Parts:
- H_MNT1, H_MNT2, H_MNT3, H_MNT4: now left out of the parts list
- TP_3V3_0, TP_5VIDEO_0: value Test Point Loop -> Test Point; footprint TestPoint:TestPoint_Loop_D1.80mm_Drill1.0mm_Beaded -> TestPoint:TestPoint_Pad_D1.0mm; now left out of the parts list
- TP_5V_0, TP_GND_0, TP_GND_1, TP_VBAT_0: value Test Point Loop -> Solder Pad; footprint TestPoint:TestPoint_Loop_D1.80mm_Drill1.0mm_Beaded -> TestPoint:TestPoint_Pad_2.5x2.5mm; Note (none) -> pad lutowniczy 2.5x2.5mm dla uzytkownika (LED/buzzer/peryfe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; now left out of the parts list
Changed lines of the file:
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@@
 		(body_style 1)
 		(exclude_from_sim no)
-		(in_bom yes)
+		(in_bom no)
 		(on_board yes)
 		(in_pos_files yes)
@@
 		(body_style 1)
 		(exclude_from_sim no)
-		(in_bom yes)
+		(in_bom no)
 		(on_board yes)
 		(in_pos_files yes)
@@
 		(body_style 1)
 		(exclude_from_sim no)
-		(in_bom yes)
+		(in_bom no)
 		(on_board yes)
 		(in_pos_files yes)
@@
 			)
 		)
-		(property "Value" "Test Point Loop"
+		(property "Value" "Solder Pad"
 			(at 75.438 148.59 90)
 			(show_name no)
@@
 			)
 		)
-		(property "Footprint" "TestPoint:TestPoint_Loop_D1.80mm_Drill1.0mm_Beaded"
+		(property "Footprint" "TestPoint:TestPoint_Pad_2.5x2.5mm"
 			(at 78.74 146.05 0)
 			(hide yes)
@@
 			)
 		)
+		(property "Note" "pad lutowniczy 2.5x2.5mm dla uzytkownika (LED/buzzer/peryferia)"
+			(at 78.74 151.13 0)
+			(hide yes)
+			(show_name no)
+			(do_not_autoplace no)
+			(effects
+				(font
+					(size 1.27 1.27)
+				)
+			)
+		)
 		(pin "1"
 		)
@@
 		(body_style 1)
 		(exclude_from_sim no)
-		(in_bom yes)
+		(in_bom no)
 		(on_board yes)
 		(in_pos_files yes)
@@
 		(body_style 1)
 		(exclude_from_sim no)
-		(in_bom yes)
+		(in_bom no)
 		(on_board yes)
 		(in_pos_files yes)
@@
 			)
 		)
-		(property "Value" "Test Point Loop"
+		(property "Value" "Solder Pad"
 			(at 75.438 156.21 90)
 			(show_name no)
@@
 			)
 		)
-		(property "Footprint" "TestPoint:TestPoint_Loop_D1.80mm_Drill1.0mm_Beaded"
+		(property "Footprint" "TestPoint:TestPoint_Pad_2.5x2.5mm"
 			(at 78.74 153.67 0)
 			(hide yes)
@@
 			)
 		)
+		(property "Note" "pad lutowniczy 2.5x2.5mm dla uzytkownika (LED/buzzer/peryferia)"
+			(at 78.74 158.75 0)
+			(hide yes)
+			(show_name no)
+			(do_not_autoplace no)
+			(effects
+				(font
+					(size 1.27 1.27)
+				)
+			)
+		)
 		(pin "1"
 		)
@@
 		(body_style 1)
 		(exclude_from_sim no)
-		(in_bom yes)
+		(in_bom no)
 		(on_board yes)
 		(in_pos_files yes)
@@
 			)
 		)
-		(property "Value" "Test Point Loop"
+		(property "Value" "Solder Pad"
 			(at 75.438 186.69 90)
 			(show_name no)
@@
 			)
 		)
-		(property "Footprint" "TestPoint:TestPoint_Loop_D1.80mm_Drill1.0mm_Beaded"
+		(property "Footprint" "TestPoint:TestPoint_Pad_2.5x2.5mm"
 			(at 78.74 184.15 0)
 			(hide yes)
@@
 			)
 		)
+		(property "Note" "pad lutowniczy 2.5x2.5mm dla uzytkownika (LED/buzzer/peryferia)"
+			(at 78.74 189.23 0)
+			(hide yes)
+			(show_name no)
+			(do_not_autoplace no)
+			(effects
+				(font
+					(size 1.27 1.27)
+				)
+			)
+		)
 		(pin "1"
 		)
@@
 		(body_style 1)
 		(exclude_from_sim no)
-		(in_bom yes)
+		(in_bom no)
 		(on_board yes)
 		(in_pos_files yes)
@@
 		(body_style 1)
 		(exclude_from_sim no)
-		(in_bom yes)
+		(in_bom no)
 		(on_board yes)
 		(in_pos_files yes)
@@
 			)
 		)
-		(property "Value" "Test Point Loop"
+		(property "Value" "Test Point"
 			(at 75.438 179.07 90)
 			(show_name no)
@@
 			)
 		)
-		(property "Footprint" "TestPoint:TestPoint_Loop_D1.80mm_Drill1.0mm_Beaded"
+		(property "Footprint" "TestPoint:TestPoint_Pad_D1.0mm"
 			(at 78.74 176.53 0)
 			(hide yes)
@@
 		(body_style 1)
 		(exclude_from_sim no)
-		(in_bom yes)
+		(in_bom no)
 		(on_board yes)
 		(in_pos_files yes)
@@
 			)
 		)
-		(property "Value" "Test Point Loop"
+		(property "Value" "Test Point"
 			(at 75.438 163.83 90)
 			(show_name no)
@@
 			)
 		)
-		(property "Footprint" "TestPoint:TestPoint_Loop_D1.80mm_Drill1.0mm_Beaded"
+		(property "Footprint" "TestPoint:TestPoint_Pad_D1.0mm"
 			(at 78.74 161.29 0)
 			(hide yes)
@@
 		(body_style 1)
 		(exclude_from_sim no)
-		(in_bom yes)
+		(in_bom no)
 		(on_board yes)
 		(in_pos_files yes)
@@
 			)
 		)
-		(property "Value" "Test Point Loop"
+		(property "Value" "Solder Pad"
 			(at 75.438 171.45 90)
 			(show_name no)
@@
 			)
 		)
-		(property "Footprint" "TestPoint:TestPoint_Loop_D1.80mm_Drill1.0mm_Beaded"
+		(property "Footprint" "TestPoint:TestPoint_Pad_2.5x2.5mm"
 			(at 78.74 168.91 0)
 			(hide yes)
@@
 			(at 78.74 173.99 0)
 			(hide yes)
+			(show_name no)
+			(do_not_autoplace no)
+			(effects
+				(font
+					(size 1.27 1.27)
+				)
+			)
+		)
+		(property "Note" "pad lutowniczy 2.5x2.5mm dla uzytkownika (LED/buzzer/peryferia)"
+			(at 78.74 173.99 0)
+			(hide yes)

Commit message: hardware: Layout improvement
Parts:
- TP_3V3_0, TP_GND_0, TP_GND_1, TP_VBAT_0: now not fitted
Changed lines of the file:
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@@
 			)
 		)
-		(property "Description" "Mounting Hole without connection 3.2mm_M3"
+		(property "Description" "Otwór montażowy M3, raster 30,5 × 30,5 mm"
 			(at 177.8 149.86 0)
 			(hide yes)
@@
 			)
 		)
-		(property "Description" "Mounting Hole without connection 3.2mm_M3"
+		(property "Description" "Otwór montażowy M3, raster 30,5 × 30,5 mm"
 			(at 177.8 154.94 0)
 			(hide yes)
@@
 			)
 		)
-		(property "Description" "test point 1mm Pad"
+		(property "Description" "Punkt pomiarowy wyjścia dzielnika napięcia pakietu — do kalibracji odczytu"
 			(at 114.3 148.59 0)
 			(hide yes)
@@
 		(exclude_from_sim no)
 		(in_bom no)
-		(on_board yes)
-		(in_pos_files yes)
-		(dnp no)
+		(on_board no)
+		(in_pos_files yes)
+		(dnp yes)
 		(fields_autoplaced yes)
 		(property "Reference" "TP_GND_1"
@@
 			)
 		)
-		(property "Description" "test point 1mm Pad"
+		(property "Description" "Drugi pad lutowniczy masy dla użytkownika"
 			(at 78.74 151.13 0)
 			(hide yes)
@@
 			)
 		)
-		(property "Description" "Mounting Hole without connection 3.2mm_M3"
+		(property "Description" "Otwór montażowy M3, raster 30,5 × 30,5 mm"
 			(at 177.8 144.78 0)
 			(hide yes)
@@
 		(exclude_from_sim no)
 		(in_bom no)
-		(on_board yes)
-		(in_pos_files yes)
-		(dnp no)
+		(on_board no)
+		(in_pos_files yes)
+		(dnp yes)
 		(fields_autoplaced yes)
 		(property "Reference" "TP_GND_0"
@@
 			)
 		)
-		(property "Description" "test point 1mm Pad"
+		(property "Description" "Pad lutowniczy masy dla użytkownika"
 			(at 78.74 158.75 0)
 			(hide yes)
@@
 		(exclude_from_sim no)
 		(in_bom no)
-		(on_board yes)
-		(in_pos_files yes)
-		(dnp no)
+		(on_board no)
+		(in_pos_files yes)
+		(dnp yes)
 		(fields_autoplaced yes)
 		(property "Reference" "TP_VBAT_0"
@@
 			)
 		)
-		(property "Description" "test point 1mm Pad"
+		(property "Description" "Pad lutowniczy VBAT dla użytkownika"
 			(at 78.74 189.23 0)
 			(hide yes)
@@
 			)
 		)
-		(property "Description" "Mounting Hole without connection 3.2mm_M3"
+		(property "Description" "Otwór montażowy M3, raster 30,5 × 30,5 mm"
 			(at 177.8 160.02 0)
 			(hide yes)
@@
 			)
 		)
-		(property "Description" "test point 1mm Pad"
+		(property "Description" "Punkt pomiarowy szyny +5V_VIDEO"
 			(at 78.74 181.61 0)
 			(hide yes)
@@
 			)
 		)
-		(property "Description" "test point 1mm Pad"
+		(property "Description" "Punkt pomiarowy przerwania z IMU — do sprawdzenia częstotliwości próbkowania na oscyloskopie"
 			(at 156.21 19.05 0)
 			(hide yes)
@@
 		(exclude_from_sim no)
 		(in_bom no)
-		(on_board yes)
-		(in_pos_files yes)
-		(dnp no)
+		(on_board no)
+		(in_pos_files yes)
+		(dnp yes)
 		(fields_autoplaced yes)
 		(property "Reference" "TP_3V3_0"
@@
 			)
 		)
-		(property "Description" "test point 1mm Pad"
+		(property "Description" "Punkt pomiarowy szyny +3V3"
 			(at 78.74 166.37 0)
 			(hide yes)
@@
 			)
 		)
-		(property "Description" "test point 1mm Pad"
+		(property "Description" "Pad lutowniczy +5 V dla użytkownika (taśma LED, buzzer, peryferia)"
 			(at 78.74 173.99 0)
 			(hide yes)

Commit message: hardware: Fixes in layout
Parts:
- TP_5V_0: now not fitted
Changed lines of the file:
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@@
 		(exclude_from_sim no)
 		(in_bom no)
-		(on_board yes)
+		(on_board no)
 		(in_pos_files yes)
-		(dnp no)
+		(dnp yes)
 		(fields_autoplaced yes)
 		(property "Reference" "TP_5V_0"

Commit message: hardware: layout checkpoint 3 - fixed DRC
Other:
- sheet Interfaces&IO ports: added USB_DN; removed USB_DM
- sheet MCU Core ports: added USB_DN; removed USB_DM
Changed lines of the file:
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@@
 			)
 		)
-		(pin "USB_DM" bidirectional
+		(pin "USB_DN" bidirectional
 			(at 134.62 76.2 0)
 			(effects
@@
 			)
 		)
-		(pin "USB_DM" bidirectional
+		(pin "USB_DN" bidirectional
 			(at 176.53 76.2 180)
 			(effects
