File: hardware/Sparrow-II/MCU.kicad_sch (KiCad schematic)
At the start: 26 parts

Commit message: hardware: VDD pins fix; OSD floating pin
Parts:
- J_SWD1: value Conn_01x04 -> Conn_01x05; footprint Connector_PinHeader_1.27mm:PinHeader_1x04_P1.27mm_Vertical_SMD_Pin1Left -> Connector_PinHeader_1.27mm:PinHeader_1x05_P1.27mm_Vertical_SMD_Pin1Left; symbol Connector_Generic:Conn_01x04 -> Connector_Generic:Conn_01x05
Connections:
- net +3V3: now also J_SWD1.1 (Pin_1), U_MCU1.19 (VDD), U_MCU1.32 (VDD), U_MCU1.48 (VDD), U_MCU1.64 (VDD)
- net GND: now also J_SWD1.5 (Pin_5); no longer J_SWD1.4 (Pin_4), U_MCU1.13 (VDDA), U_MCU1.19 (VDD), U_MCU1.32 (VDD), U_MCU1.48 (VDD), U_MCU1.64 (VDD)
- net NRST: now also J_SWD1.4 (Pin_4); no longer J_SWD1.3 (Pin_3)
- net SWCLK: now also J_SWD1.3 (Pin_3); no longer J_SWD1.2 (Pin_2)
- net SWDIO: now also J_SWD1.2 (Pin_2); no longer J_SWD1.1 (Pin_1)
- net at C_VDDA1.1, C_VDDA_HF1.1, FB_VDDA1.2: now also U_MCU1.13 (VDDA)
Other:
- moved on the sheet: C_VDD1, C_VDD2, C_VDD3, C_VDD4, C_VDDA1, C_VDDA_HF1, C_VDD_BULK1, FB_VDDA1

Commit message: hardware: change in oscilator values
Parts:
- C_HSE1, C_HSE2: value 27pF -> 12pF
- R_HSE2: value 1k -> 0R
- Y_HSE1: value 8MHz -> 8MHz CL=10pF ESR<150R
Changed lines of the file:
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@@
 	(wire
 		(pts
+			(xy 97.79 120.65) (xy 97.79 118.11)
+		)
+		(stroke
+			(width 0)
+			(type default)
+		)
+	)
+	(wire
+		(pts
 			(xy 262.89 138.43) (xy 271.78 138.43)
 		)
@@
 			)
 		)
-		(property "Value" "27pF"
+		(property "Value" "12pF"
 			(at 83.82 59.69 90)
 			(show_name no)
@@
 			)
 		)
-		(property "Value" "1k"
+		(property "Value" "0R"
 			(at 107.95 60.96 90)
 			(show_name no)
@@
 	)
 	(symbol
+		(lib_id "power:+3V3")
+		(at 97.79 118.11 0)
+		(unit 1)
+		(body_style 1)
+		(exclude_from_sim no)
+		(in_bom yes)
+		(on_board yes)
+		(in_pos_files yes)
+		(dnp no)
+		(property "Reference" "#PWR040"
+			(at 97.79 114.935 0)
+			(hide yes)
+			(show_name no)
+			(do_not_autoplace no)
+			(effects
+				(font
+					(size 1.27 1.27)
+				)
+			)
+		)
+		(property "Value" "+3V3"
+			(at 94.488 118.11 0)
+			(show_name no)
+			(do_not_autoplace no)
+			(effects
+				(font
+					(size 1.27 1.27)
+				)
+			)
+		)
+		(property "Footprint" ""
+			(at 97.79 118.11 0)
+			(hide yes)
+			(show_name no)
+			(do_not_autoplace no)
+			(effects
+				(font
+					(size 1.27 1.27)
+				)
+			)
+		)
+		(property "Datasheet" ""
+			(at 97.79 118.11 0)
+			(hide yes)
+			(show_name no)
+			(do_not_autoplace no)
+			(effects
+				(font
+					(size 1.27 1.27)
+				)
+			)
+		)
+		(property "Description" "Power symbol"
+			(at 97.79 118.11 0)
+			(hide yes)
+			(show_name no)
+			(do_not_autoplace no)
+			(effects
+				(font
+					(size 1.27 1.27)
+				)
+			)
+		)
+		(pin "1"
+		)
+		(instances
+			(project "Flight Controller"
+				(path "/64d08664-7c2b-4b48-a9dd-dae3f797396a/68c3808c-080f-4420-8614-2f4fdfbceec8"
+					(reference "#PWR040")
+					(unit 1)
+				)
+			)
+		)
+	)
+	(symbol
 		(lib_id "Device:LED")
 		(at 127 204.47 90)
@@
 			)
 		)
-		(property "Value" "27pF"
+		(property "Value" "12pF"
 			(at 83.82 46.99 90)
 			(show_name no)
@@
 			)
 		)
-		(property "Value" "8MHz"
+		(property "Value" "8MHz CL=10pF ESR<150R"
 			(at 104.14 56.0068 90)
 			(show_name no)
@@
 					(unit 1)
 				)
-			)
-		)
-	)
-	(wire
-		(pts
-			(xy 97.79 120.65) (xy 97.79 118.11)
-		)
-		(stroke
-			(width 0)
-			(type default)
-		)
-	)
-	(symbol
-		(lib_id "power:+3V3")
-		(at 97.79 118.11 0)
-		(unit 1)
-		(body_style 1)
-		(exclude_from_sim no)
-		(in_bom yes)
-		(on_board yes)
-		(in_pos_files yes)
-		(dnp no)
-		(fields_autoplaced yes)
-		(property "Reference" "#PWR040"
-			(at 97.79 114.935 0)
-			(hide yes)
-			(show_name no)
-			(do_not_autoplace no)
-			(effects
-				(font
-					(size 1.27 1.27)
-				)
-			)
-		)
-		(property "Value" "+3V3"
-			(at 97.79 121.285 0)
-			(show_name no)
-			(do_not_autoplace no)
-			(effects
-				(font
-					(size 1.27 1.27)
-				)
-			)
-		)
-		(property "Footprint" ""
-			(at 97.79 118.11 0)
-			(hide yes)
-			(show_name no)
-			(do_not_autoplace no)
-			(effects
-				(font
-					(size 1.27 1.27)
-				)
-			)
-		)
-		(property "Datasheet" ""
-			(at 97.79 118.11 0)
-			(hide yes)
-			(show_name no)
-			(do_not_autoplace no)
-			(effects
-				(font
-					(size 1.27 1.27)
-				)
-			)
-		)
-		(property "Description" "Power symbol"
-			(at 97.79 118.11 0)
-			(hide yes)
-			(show_name no)
-			(do_not_autoplace no)
-			(effects
-				(font
-					(size 1.27 1.27)
-				)
-			)
-		)
-		(pin "1"
-		)
-		(instances
-			(project "Flight Controller"
-				(path "/64d08664-7c2b-4b48-a9dd-dae3f797396a/68c3808c-080f-4420-8614-2f4fdfbceec8"
-					(reference "#PWR040")
-					(unit 1)
-				)

Commit message: hardware: BOM actualization and second layout
Parts:
- C_HSE1, C_HSE2: footprint Capacitor_SMD:C_0402_1005Metric_Pad0.74x0.62mm_HandSolder -> Capacitor_SMD:C_0402_1005Metric; Dielectric (none) -> C0G/NP0; Voltage (none) -> 50V
- C_NRST1, C_VDD1, C_VDD2, C_VDD3, C_VDD4, C_VDDA1, C_VDDA_HF1: footprint Capacitor_SMD:C_0402_1005Metric_Pad0.74x0.62mm_HandSolder -> Capacitor_SMD:C_0402_1005Metric; Dielectric (none) -> X7R; Voltage (none) -> 16V
- C_VCAP1: footprint Capacitor_SMD:C_0805_2012Metric_Pad1.18x1.45mm_HandSolder -> Capacitor_SMD:C_0805_2012Metric; Dielectric (none) -> X5R; Voltage (none) -> 10V
- C_VDD_BULK1: footprint Capacitor_SMD:C_0402_1005Metric_Pad0.74x0.62mm_HandSolder -> Capacitor_SMD:C_0603_1608Metric; Dielectric (none) -> X7R; Voltage (none) -> 16V
- FB_VDDA1: footprint Inductor_SMD:L_0402_1005Metric_Pad0.77x0.64mm_HandSolder -> Inductor_SMD:L_0402_1005Metric; Spec (none) -> 100R@100MHz, Idc>=100mA
- JP_BOOT0: now left out of the parts list
- J_SWD1: value Conn_01x05 -> SWD Pads; footprint Connector_PinHeader_1.27mm:PinHeader_1x05_P1.27mm_Vertical_SMD_Pin1Left -> SparrowHawk:SolderPads_SWD_1x05; Note (none) -> Pady lutownicze zamiast zlacza: 3V3 / SWDIO / SWCLK / NRST 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; now left out of the parts list
- LED_PWR1: footprint LED_SMD:LED_0603_1608Metric_Pad1.05x0.95mm_HandSolder -> LED_SMD:LED_0603_1608Metric; Spec (none) -> green, If=1.5mA @3.3V via R_LED1
- LED_STAT1: footprint LED_SMD:LED_0603_1608Metric_Pad1.05x0.95mm_HandSolder -> LED_SMD:LED_0603_1608Metric; Spec (none) -> blue
- LED_STAT2: footprint LED_SMD:LED_0603_1608Metric_Pad1.05x0.95mm_HandSolder -> LED_SMD:LED_0603_1608Metric; Spec (none) -> red
- R_BOOT0, R_HSE2, R_I2C_SCL1, R_I2C_SDA1, R_LED1, R_LED2, R_LED3: footprint Resistor_SMD:R_0402_1005Metric_Pad0.72x0.64mm_HandSolder -> Resistor_SMD:R_0402_1005Metric; Power (none) -> 0.063W; Tolerance (none) -> 1%
- U_MCU1: MPN (none) -> STM32F722RET6; Manufacturer (none) -> STMicroelectronics
- Y_HSE1: footprint Crystal:Crystal_SMD_3225-4Pin_3.2x2.5mm_HandSoldering -> Crystal:Crystal_SMD_3225-4Pin_3.2x2.5mm; Spec (none) -> 8MHz, CL=10pF, ESR<=150R, 3225 4-pad (C_HSE1/2=12pF C0G)

Commit message: hardware: Layout improvement
Parts:
- FB_VDDA1: Spec 100R@100MHz, Idc>=100mA -> 100 Ω @ 100 MHz, Idc ≥ 100 mA
- LED_PWR1: Spec green, If=1.5mA @3.3V via R_LED1 -> zielona, 0603, If ≈ 1,5 mA przy 3,3 V
- LED_STAT1: Spec blue -> niebieska, 0603
- LED_STAT2: Spec red -> czerwona, 0603
- Y_HSE1: Spec 8MHz, CL=10pF, ESR<=150R, 3225 4-pad (C_HSE1/2=12pF C0G) -> 8 MHz, CL = 10 pF, ESR ≤ 150 Ω, obudowa 3225 4-pad (C_HSE1/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
Changed lines of the file:
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@@
 			)
 		)
-		(property "Description" "Generic connector, single row, 01x04, script generated (kicad-library-utils/schlib/autogen/connector/)"
+		(property "Description" "Pady programowania SWD: 3V3 / SWDIO / SWCLK / NRST / GND. Napięcie odniesienia obowiązkowe, bez niego ST-Link nie ustawi translatorów poziomów"
 			(at 102.87 125.73 0)
 			(hide yes)
@@
 			)
 		)
-		(property "Description" "Light emitting diode"
+		(property "Description" "Dioda sygnalizacji zasilania +3V3"
 			(at 74.93 204.47 0)
 			(hide yes)
@@
 			)
 		)
-		(property "Spec" "green, If=1.5mA @3.3V via R_LED1"
+		(property "Spec" "zielona, 0603, If ≈ 1,5 mA przy 3,3 V"
 			(at 74.93 204.47 0)
 			(hide yes)
@@
 			)
 		)
-		(property "Description" "Resistor"
+		(property "Description" "Podciągnięcie linii danych I2C1"
 			(at 363.22 167.64 0)
 			(hide yes)
@@
 			)
 		)
-		(property "Description" "Unpolarized capacitor"
+		(property "Description" "Kondensator obciążenia kwarcu 8 MHz. C0G obowiązkowo — na X7R pojemność dryfuje i rozstraja oscylator"
 			(at 83.82 64.77 0)
 			(hide yes)
@@
 			)
 		)
-		(property "Description" "Resistor"
+		(property "Description" "Rezystor szeregowy oscylatora MCU, 0 Ω. Zostawiony jako miejsce na ograniczenie mocy wzbudzenia kwarcu"
 			(at 107.95 64.77 0)
 			(hide yes)
@@
 			)
 		)
-		(property "Description" "Unpolarized capacitor"
+		(property "Description" "Odsprzęganie zasilania analogowego VDDA"
 			(at 257.81 97.79 0)
 			(hide yes)
@@
 			)
 		)
-		(property "Description" "Light emitting diode"
+		(property "Description" "Dioda statusu sterowana z PB1"
 			(at 127 204.47 0)
 			(hide yes)
@@
 			)
 		)
-		(property "Spec" "red"
+		(property "Spec" "czerwona, 0603"
 			(at 127 204.47 0)
 			(hide yes)
@@
 			)
 		)
-		(property "Description" "Unpolarized capacitor"
+		(property "Description" "Kondensator wewnętrznego regulatora rdzenia 1,2 V. Wartość narzucona przez datasheet STM32F722 (LQFP64, jeden pin VCAP)"
 			(at 210.82 182.88 0)
 			(hide yes)
@@
 			)
 		)
-		(property "Description" "Unpolarized capacitor"
+		(property "Description" "Drugi kondensator obciążenia kwarcu 8 MHz"
 			(at 83.82 52.07 0)
 			(hide yes)
@@
 			)
 		)
-		(property "Description" "Ferrite bead"
+		(property "Description" "Koralik ferrytowy oddzielający zasilanie analogowe VDDA od cyfrowego +3V3 — obniża szum na ADC"
 			(at 280.67 91.44 0)
 			(hide yes)
@@
 			)
 		)
-		(property "Spec" "100R@100MHz, Idc>=100mA"
+		(property "Spec" "100 Ω @ 100 MHz, Idc ≥ 100 mA"
 			(at 280.67 91.44 0)
 			(hide yes)
@@
 			)
 		)
-		(property "Description" "Unpolarized capacitor"
+		(property "Description" "Odsprzęganie pinu VDD procesora"
 			(at 293.37 72.39 0)
 			(hide yes)
@@
 			)
 		)
-		(property "Description" "STMicroelectronics Arm Cortex-M7 MCU, 512KB flash, 256KB RAM, 216 MHz, 1.7-3.6V, 50 GPIO, LQFP64"
+		(property "Description" "Procesor główny. Cortex-M7 216 MHz, 512 kB Flash, 256 kB RAM — target Betaflight/INAV"
 			(at 242.57 156.21 0)
 			(hide yes)
@@
 			)
 		)
-		(property "Description" "Resistor"
+		(property "Description" "Rezystor ograniczający prąd diody zasilania"
 			(at 74.93 190.5 0)
 			(hide yes)
@@
 			)
 		)
-		(property "Description" "Jumper, 2-pole, open"
+		(property "Description" "Zworka lutownicza BOOT0 → +3V3. Zwarcie wymusza start bootloadera DFU"
 			(at 189.23 115.57 0)
 			(hide yes)
@@
 			)
 		)
-		(property "Description" "Unpolarized capacitor"
+		(property "Description" "Odsprzęganie pinu VDD procesora"
 			(at 265.43 72.39 0)
 			(hide yes)
@@
 			)
 		)
-		(property "Description" "Four pin crystal, GND on pins 2 and 4"
+		(property "Description" "Kwarc zegara głównego. Wymagany — STM32F722 nie ma HSI48 ani CRS, więc bez niego USB nie wystartuje"
 			(at 96.52 58.42 0)
 			(hide yes)
@@
 			)
 		)
-		(property "Spec" "8MHz, CL=10pF, ESR<=150R, 3225 4-pad (C_HSE1/2=12pF C0G)"
+		(property "Spec" "8 MHz, CL = 10 pF, ESR ≤ 150 Ω, obudowa 3225 4-pad (C_HSE1/2 = 12 pF C0G)"
 			(at 96.52 58.42 0)
 			(hide yes)
@@
 			)
 		)
-		(property "Description" "Resistor"
+		(property "Description" "Rezystor ograniczający prąd diody statusu 1"
 			(at 101.6 190.5 0)
 			(hide yes)
@@
 			)
 		)
-		(property "Description" "Unpolarized capacitor"
+		(property "Description" "Odsprzęganie HF zasilania analogowego VDDA"
 			(at 271.78 97.79 0)
 			(hide yes)
@@
 			)
 		)
-		(property "Description" "Unpolarized capacitor"
+		(property "Description" "Odsprzęganie pinu VDD procesora — jeden na każdą parę pinów zasilania"
 			(at 250.19 72.39 0)
 			(hide yes)
@@
 			)
 		)
-		(property "Description" "Unpolarized capacitor"
+		(property "Description" "Filtr linii resetu — tłumi zakłócenia i wydłuża impuls startowy"
 			(at 208.28 107.95 0)
 			(hide yes)
@@
 			)
 		)
-		(property "Description" "Resistor"
+		(property "Description" "Podciągnięcie linii zegara I2C1 — magistrala barometru i kompasu w module GPS"
 			(at 363.22 148.59 0)
 			(hide yes)
@@
 			)
 		)
-		(property "Description" "Unpolarized capacitor"
+		(property "Description" "Odsprzęganie pinu VDD procesora"
 			(at 279.4 72.39 0)
 			(hide yes)
@@
 			)
 		)
-		(property "Description" "Light emitting diode"
+		(property "Description" "Dioda statusu sterowana z PB0"
 			(at 101.6 204.47 0)
 			(hide yes)
@@
 			)
 		)
-		(property "Spec" "blue"
+		(property "Spec" "niebieska, 0603"
 			(at 101.6 204.47 0)
 			(hide yes)
@@
 			)
 		)
-		(property "Description" "Unpolarized capacitor"
+		(property "Description" "Lokalny zapas ładunku szyny VDD procesora"
 			(at 308.61 72.39 0)
 			(hide yes)
@@
 			)
 		)
-		(property "Description" "Resistor"
+		(property "Description" "Rezystor ściągający BOOT0 do masy. Domyślnie start z pamięci Flash"
 			(at 189.23 124.46 0)
 			(hide yes)
@@
 			)
 		)
-		(property "Description" "Resistor"
+		(property "Description" "Rezystor ograniczający prąd diody statusu 2"
 			(at 127 190.5 0)
 			(hide yes)

Commit message: hardware: layout checkpoint 3 - fixed DRC
Connections:
- net USB_DM renamed USB_DN
Changed lines of the file:
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@@
 		)
 	)
-	(hierarchical_label "USB_DM"
+	(hierarchical_label "USB_DN"
 		(shape bidirectional)
 		(at 271.78 143.51 0)
