File: hardware/Sparrow-II/Sensors.kicad_sch (KiCad schematic)
At the start: 14 parts

Commit message: hardware: fixes connected to ERC errors 1/2
Parts:
- U_BARO1: footprint FC Drone Footprint Library:XDCR_DPS310 -> SparrowHawk:XDCR_DPS310
- U_IMU1: footprint FC Drone Footprint Library:PQFN50P300X250X97-14N -> SparrowHawk:PQFN50P300X250X97-14N
Changed lines of the file:
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@@
 			)
 		)
-		(property "Footprint" "FC Drone Footprint Library:XDCR_DPS310"
+		(property "Footprint" "SparrowHawk:XDCR_DPS310"
 			(at 137.16 168.91 0)
 			(hide yes)
@@
 			)
 		)
-		(property "Footprint" "FC Drone Footprint Library:PQFN50P300X250X97-14N"
+		(property "Footprint" "SparrowHawk:PQFN50P300X250X97-14N"
 			(at 114.3 86.36 0)
 			(hide yes)

Commit message: hardware: VDD pins fix; OSD floating pin
Connections:
- net GND: now also U_IMU1.7 (RESV_7)
- no-connect marks 6 -> 5
Changed lines of the file:
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@@
 	)
 	(no_connect
-		(at 139.7 96.52)
-	)
-	(no_connect
 		(at 139.7 91.44)
 	)
@@
 	)
 	(no_connect
-		(at 88.9 81.28)
-	)
-	(no_connect
 		(at 139.7 88.9)
 	)
@@
 		)
 	)
+	(wire
+		(pts
+			(xy 139.7 96.52) (xy 144.78 96.52)
+		)
+		(stroke
+			(width 0)
+			(type default)
+		)
+	)
+	(wire
+		(pts
+			(xy 144.78 96.52) (xy 144.78 101.6)
+		)
+		(stroke
+			(width 0)
+			(type default)
+		)
+	)
+	(junction
+		(at 144.78 101.6)
+		(diameter 0)
+		(color 0 0 0 0)
+	)
+	(no_connect
+		(at 88.9 81.28)
+	)
 )

Commit message: hardware: BOM actualization and second layout
Parts:
- C_BARO1, C_BARO2, C_FLASH1, C_IMU_VDD2, C_IMU_VIO1, C_IMU_VIO2: footprint Capacitor_SMD:C_0402_1005Metric_Pad0.74x0.62mm_HandSolder -> Capacitor_SMD:C_0402_1005Metric; Dielectric (none) -> X7R; Voltage (none) -> 16V
- C_IMU_VDD1: footprint Capacitor_SMD:C_0402_1005Metric_Pad0.74x0.62mm_HandSolder -> Capacitor_SMD:C_0402_1005Metric; Dielectric (none) -> X5R; Voltage (none) -> 16V
- FB_IMU1: Spec (none) -> 600R@100MHz, Idc>=200mA
- R_FLASH_CS1, R_FLASH_HD1, R_FLASH_WP1: footprint Resistor_SMD:R_0402_1005Metric_Pad0.72x0.64mm_HandSolder -> Resistor_SMD:R_0402_1005Metric; Power (none) -> 0.063W; Tolerance (none) -> 1%
- U_BARO1: AVAILABILITY Unavailable -> (none); Availability In Stock -> (none); Check_prices https://www.snapeda.com/parts/DPS310/Infineon/view-part/?re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 -> (none); Description_1 Pressure Sensor 4.35PSI ~ 17.4PSI (30kPa ~ 120kPa) Vented G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 -> (none); MF Infineon Technologies -> (none); MP DPS310 -> (none); MPN (none) -> DPS310; Manufacturer (none) -> Infineon Technologies; PRICE None -> (none); Price None -> (none); SnapEDA_Link https://www.snapeda.com/parts/DPS310/Infineon/view-part/?re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 -> (none)
- U_FLASH1: MPN (none) -> W25Q128JVEIQ; Manufacturer (none) -> Winbond; Note (none) -> kod obudowy E = WSON 8x6mm. Wariant P = WSON 6x5mm oszczedz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; Spec (none) -> 128Mbit SPI NOR, 2.7-3.6V
- U_IMU1: Availability In Stock -> (none); Check_prices https://www.snapeda.com/parts/ICM-42688-P/TDK+InvenSense/vi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 -> (none); Description_1 Accelerometer, Gyroscope, 6 Axis Sensor - Output -> (none); MANUFACTURER TDK InvenSense -> (none); MAXIMUM_PACKAGE_HEIGHT 0.97mm -> (none); MF TDK InvenSense -> (none); MP ICM-42688-P -> (none); MPN (none) -> ICM-42688-P; Manufacturer (none) -> TDK InvenSense; PARTREV 1.2 -> (none); Price None -> (none); STANDARD IPC-7351B -> (none); SnapEDA_Link https://www.snapeda.com/parts/ICM-42688-P/TDK+InvenSense/vi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 -> (none)

Commit message: hardware: Layout improvement
Parts:
- FB_IMU1: Spec 600R@100MHz, Idc>=200mA -> 600 Ω @ 100 MHz, Idc ≥ 200 mA
- U_FLASH1: Spec 128Mbit SPI NOR, 2.7-3.6V -> 128 Mbit SPI NOR, 2,7–3,6 V
Changed lines of the file:
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@@
 			)
 		)
-		(property "Description" "Resistor"
+		(property "Description" "Podciągnięcie /WP — wyłącza sprzętową blokadę zapisu"
 			(at 257.81 90.17 0)
 			(hide yes)
@@
 			)
 		)
-		(property "Description" "Unpolarized capacitor"
+		(property "Description" "Drugi kondensator odsprzęgający VDDIO wg noty aplikacyjnej TDK"
 			(at 177.8 96.52 0)
 			(hide yes)
@@
 			)
 		)
-		(property "Description" "Unpolarized capacitor"
+		(property "Description" "Odsprzęganie zasilania analogowego IMU"
 			(at 160.02 85.09 0)
 			(hide yes)
@@
 			)
 		)
-		(property "Description" "128Mbit / 16MiB Serial Flash Memory, Standard/Dual/Quad SPI, 2.7-3.6V, WSON-8"
+		(property "Description" "Pamięć Flash SPI 16 MB na logi blackbox"
 			(at 303.53 64.77 0)
 			(hide yes)
@@
 			)
 		)
-		(property "Spec" "128Mbit SPI NOR, 2.7-3.6V"
+		(property "Spec" "128 Mbit SPI NOR, 2,7–3,6 V"
 			(at 303.53 92.71 0)
 			(hide yes)
@@
 			)
 		)
-		(property "Description" "Unpolarized capacitor"
+		(property "Description" "Odsprzęganie zasilania interfejsu cyfrowego IMU"
 			(at 160.02 96.52 0)
 			(hide yes)
@@
 			)
 		)
-		(property "Description" "Unpolarized capacitor"
+		(property "Description" "Odsprzęganie VDDIO barometru"
 			(at 167.64 166.37 0)
 			(hide yes)
@@
 			)
 		)
-		(property "Description" "Ferrite bead"
+		(property "Description" "Koralik ferrytowy na zasilaniu IMU — odcina szum przetwornicy od czujnika"
 			(at 163.83 73.66 0)
 			(hide yes)
@@
 			)
 		)
-		(property "Spec" "600R@100MHz, Idc>=200mA"
+		(property "Spec" "600 Ω @ 100 MHz, Idc ≥ 200 mA"
 			(at 163.83 73.66 0)
 			(hide yes)
@@
 			)
 		)
-		(property "Datasheet" ""
+		(property "Datasheet" "https://www.infineon.com/dgdl/Infineon-DPS310-DataSheet-v01_02-EN.pdf"
 			(at 137.16 168.91 0)
 			(hide yes)
@@
 			)
 		)
-		(property "Description" "The DPS310 is a miniaturized Digital Barometric Air Pressure Sensor with a high accuracy and a low current consumption, capable of measuring both pressure and temperature."
+		(property "Description" "Barometr. Interfejs I2C wybrany przez CSB→VDDIO, adres 0x76 przez SDO→GND"
 			(at 137.16 168.91 0)
 			(hide yes)
@@
 			)
 		)
-		(property "Description" "Unpolarized capacitor"
+		(property "Description" "Odsprzęganie zasilania pamięci Flash"
 			(at 321.31 78.74 0)
 			(hide yes)
@@
 			)
 		)
-		(property "Description" "Unpolarized capacitor"
+		(property "Description" "Odsprzęganie zasilania barometru"
 			(at 152.4 166.37 0)
 			(hide yes)
@@
 			)
 		)
-		(property "Description" "Resistor"
+		(property "Description" "Podciągnięcie /HOLD — wyłącza wstrzymywanie transmisji"
 			(at 241.3 90.17 0)
 			(hide yes)
@@
 			)
 		)
-		(property "Datasheet" ""
+		(property "Datasheet" "https://invensense.tdk.com/wp-content/uploads/2020/03/DS-000347-ICM-42688-P-v1.5.pdf"
 			(at 114.3 86.36 0)
 			(hide yes)
@@
 			)
 		)
-		(property "Description" ""
+		(property "Description" "Żyroskop i akcelerometr 6-osiowy, SPI. Główny czujnik pętli sterowania"
 			(at 114.3 86.36 0)
 			(hide yes)
@@
 			)
 		)
-		(property "Description" "Resistor"
+		(property "Description" "Podciągnięcie /CS pamięci — trzyma układ nieaktywny, zanim MCU skonfiguruje piny"
 			(at 287.02 80.01 0)
 			(hide yes)
@@
 			)
 		)
-		(property "Description" "Unpolarized capacitor"
+		(property "Description" "Odsprzęganie HF zasilania IMU"
 			(at 177.8 85.09 0)
 			(hide yes)
