File: hardware/Sparrow-II/Power.kicad_sch (KiCad schematic)
At the start: 34 parts

Commit message: hardware: fixes connected to ERC errors 1/2
Parts:
- J_BAT1: footprint FC Drone Footprint Library:VBAT_SolderPad_2x_5x5mm -> SparrowHawk:VBAT_SolderPad_2x_5x5mm
- Q_RPP1: footprint FC Drone Footprint Library:SOT23_INF-M -> SparrowHawk:SOT23_INF-M
- U_BUCK1: footprint FC Drone Footprint Library:SOIC127P600X170-9N -> SparrowHawk:SOIC127P600X170-9N; Description_1 SIMPLE SWITCHER® 40-V, 3.5-A, 2.2-MHz step-down converter w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 -> (none)
Connections:
- net EXP renamed GND

Commit message: hardware: OSD quick fixes
Changed lines of the file:
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@@
 	)
 	(junction
+		(at 304.8 111.76)
+		(diameter 0)
+		(color 0 0 0 0)
+	)
+	(junction
 		(at 77.47 127)
 		(diameter 0)
@@
 	(wire
 		(pts
+			(xy 304.8 106.68) (xy 304.8 111.76)
+		)
+		(stroke
+			(width 0)
+			(type default)
+		)
+	)
+	(wire
+		(pts
 			(xy 49.53 73.66) (xy 57.15 73.66)
 		)
@@
 					(unit 1)
 				)
+			)
+		)
+	)
+	(symbol
+		(lib_id "power:PWR_FLAG")
+		(at 304.8 106.68 0)
+		(unit 1)
+		(body_style 1)
+		(exclude_from_sim no)
+		(in_bom no)
+		(on_board no)
+		(in_pos_files no)
+		(dnp no)
+		(fields_autoplaced yes)
+		(property "Reference" "#FLG07"
+			(at 304.8 104.775 0)
+			(hide yes)
+			(show_name no)
+			(do_not_autoplace no)
+			(effects
+				(font
+					(size 1.27 1.27)
+				)
+			)
+		)
+		(property "Value" "PWR_FLAG"
+			(at 304.8 103.505 0)
+			(show_name no)
+			(do_not_autoplace no)
+			(effects
+				(font
+					(size 1.27 1.27)
+				)
+			)
+		)
+		(property "Footprint" ""
+			(at 304.8 106.68 0)
+			(hide yes)
+			(show_name no)
+			(do_not_autoplace no)
+			(effects
+				(font
+					(size 1.27 1.27)
+				)
+			)
+		)
+		(property "Datasheet" ""
+			(at 304.8 106.68 0)
+			(hide yes)
+			(show_name no)
+			(do_not_autoplace no)
+			(effects
+				(font
+					(size 1.27 1.27)
+				)
+			)
+		)
+		(property "Description" "Special symbol for telling ERC where power comes from"
+			(at 304.8 106.68 0)
+			(hide yes)
+			(show_name no)
+			(do_not_autoplace no)
+			(effects
+				(font
+					(size 1.27 1.27)
+				)
+			)
+		)
+		(pin "1"
+		)
+		(instances
+			(project "Flight Controller"
+				(path "/64d08664-7c2b-4b48-a9dd-dae3f797396a/591bf136-b725-40d6-a933-58d61d366558"
+					(reference "#FLG07")
+					(unit 1)
+				)

Commit message: hardware: BOM actualization and second layout
Parts:
- C_3V3_BULK1, C_5V_BULK1: footprint Capacitor_SMD:C_0603_1608Metric_Pad1.08x0.95mm_HandSolder -> Capacitor_SMD:C_0603_1608Metric; Dielectric (none) -> X5R; Voltage (none) -> 16V
- C_B1: value 470uF -> 100uF; footprint Capacitor_SMD:CP_Elec_8x6.9 -> Capacitor_SMD:CP_Elec_6.3x7.7; MPN (none) -> EEE-FTH101XAP; Manufacturer (none) -> Panasonic; Note (none) -> bulk VBAT; TI SNVSA81B zaleca 47-100uF. ESR 340mR tlumi dzw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; Voltage (none) -> 50V
- C_B2: footprint Capacitor_SMD:C_1210_3225Metric_Pad1.33x2.70mm_HandSolder -> Capacitor_SMD:C_1210_3225Metric; Note (none) -> Wylaczony: redundantny z C_BUCK_IN1/2 (ta sama siec VBAT); now not fitted; now left out of the parts list
- C_B3: footprint Capacitor_SMD:C_0603_1608Metric_Pad1.08x0.95mm_HandSolder -> Capacitor_SMD:C_0603_1608Metric; Note (none) -> Wylaczony: redundantny z C_BUCK_IN1/2; now not fitted; now left out of the parts list
- C_B4: footprint Capacitor_SMD:C_0402_1005Metric_Pad0.74x0.62mm_HandSolder -> Capacitor_SMD:C_0402_1005Metric; Note (none) -> Wylaczony: redundantny z C_BUCK_IN3; now not fitted; now left out of the parts list
- C_BUCK_BOOT1: Dielectric (none) -> X7R; Voltage (none) -> 50V
- C_BUCK_IN1: value 2.2uF -> 4.7uF; footprint Capacitor_SMD:C_1210_3225Metric_Pad1.33x2.70mm_HandSolder -> Capacitor_SMD:C_1210_3225Metric; Dielectric (none) -> X7R; Note (none) -> 100V wg TI SNVSA81B (2x Vin); przy 25V bias ok. 2uF efektyw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; Voltage (none) -> 100V
- C_BUCK_IN2: value 2.2uF -> 4.7uF; footprint Capacitor_SMD:C_1210_3225Metric_Pad1.33x2.70mm_HandSolder -> Capacitor_SMD:C_1210_3225Metric; Dielectric (none) -> X7R; Voltage (none) -> 100V
- C_BUCK_IN3: footprint Capacitor_SMD:C_0402_1005Metric_Pad0.74x0.62mm_HandSolder -> Capacitor_SMD:C_0603_1608Metric; Dielectric (none) -> X7R; Voltage (none) -> 100V
- C_BUCK_OUT1: footprint Capacitor_SMD:C_1210_3225Metric_Pad1.33x2.70mm_HandSolder -> Capacitor_SMD:C_1210_3225Metric; Dielectric (none) -> X5R; Voltage (none) -> 16V
- C_BUCK_OUT2: footprint Capacitor_SMD:C_1210_3225Metric_Pad1.33x2.70mm_HandSolder -> Capacitor_SMD:C_1210_3225Metric; Note (none) -> Wylaczony: 1x47uF wystarcza przy 0,8 A (ripple ~12 mV); now not fitted; now left out of the parts list
- C_BUCK_SS1, C_LDO_IN1, C_LDO_OUT1, C_VBAT_ADC1, C_VID3: footprint Capacitor_SMD:C_0402_1005Metric_Pad0.74x0.62mm_HandSolder -> Capacitor_SMD:C_0402_1005Metric; Dielectric (none) -> X7R; Voltage (none) -> 16V
- C_VID1: footprint Capacitor_SMD:C_0805_2012Metric_Pad1.18x1.45mm_HandSolder -> Capacitor_SMD:C_0805_2012Metric; Dielectric (none) -> X5R; Voltage (none) -> 16V
- C_VID2: footprint Capacitor_SMD:C_0805_2012Metric_Pad1.18x1.45mm_HandSolder -> Capacitor_SMD:C_0805_2012Metric; Note (none) -> Wylaczony: 1x22uF wystarcza dla kamery; usuwa tez blad symb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; now not fitted; now left out of the parts list
- D_BUCK1: value B560C-13-F -> B260A-13-F; footprint Diode_SMD:D_SMB -> Diode_SMD:D_SMA; MPN (none) -> B260A-13-F; Manufacturer (none) -> Diodes Incorporated; Note (none) -> 60V/2A. Poprzednio B560C-13-F (5A) w footprincie SMB - B560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
- D_TVS1: MPN (none) -> SMAJ28A; Manufacturer (none) -> Littelfuse; Note (none) -> Vwm 28V, Vc 45.4V @8.8A. Uwaga: LMR14030 ma abs.max VIN = 4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
- J_BAT1: Note (none) -> Awaryjne wejscie VBAT (pakiet lutowany wprost). Nie uzywac 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
- L_BUCK1: Note (none) -> SRN6028 zostaje - zapas na nasycenie przy zwarciu +5V. SRN5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; Spec (none) -> 6.8uH, Isat>=2.5A, Irms>=1.5A, DCR<=80mOhm
- L_VID1: footprint Inductor_SMD:L_Wuerth_WE-PD-Typ-7345 -> Inductor_SMD:L_Sunlord_SWPA3015S; MPN (none) -> SWPA3015S4R7MT; Manufacturer (none) -> Sunlord; Note (none) -> 3x3x1.5mm, 1.09A, DCR 163mR. Poprzednio WE-PD 7345 (7.3x4.5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
- Q_RPP1: symbol 2026-04-23_12-45-33:IRLML6402TRPBF -> SparrowHawk_Misc:IRLML6402TRPBF
- R_BUCK_FB1, R_BUCK_FB2, R_BUCK_RT1, R_RPP1, R_VBAT_D1, R_VBAT_D2: footprint Resistor_SMD:R_0402_1005Metric_Pad0.72x0.64mm_HandSolder -> Resistor_SMD:R_0402_1005Metric; Power (none) -> 0.063W; Tolerance (none) -> 1%
- U_BUCK1: Availability In Stock -> (none); Check_prices https://www.snapeda.com/parts/LMR14030SDDAR/Texas+Instrumen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 -> (none); MANUFACTURER Texas Instruments -> (none); MAXIMUM_PACKAGE_HEIGHT 1.70 mm -> (none); MF Texas Instruments -> (none); MP LMR14030SDDAR -> (none); MPN (none) -> LMR14030SDDAR; Manufacturer (none) -> Texas Instruments; PARTREV A -> (none); Price None -> (none); Purchase-URL https://www.snapeda.com/api/url_track_click_mouser/?unipart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 -> (none); STANDARD IPC 7351B -> (none); SnapEDA_Link https://www.snapeda.com/parts/LMR14030SDDAR/Texas+Instrumen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 -> (none)
- U_LDO1: footprint Package_TO_SOT_SMD:SOT-23-5_HandSoldering -> Package_TO_SOT_SMD:SOT-23-5; Availability In Stock -> (none); Check_prices https://www.snapeda.com/parts/AP2112K-3.3TRG1/Diodes+Inc./v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 -> (none); Description_1 Voltage Regulators, LDO, 600mA CMOS LDO 50mA 3.3V 250mV | D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 -> (none); MANUFACTURER Diodes Inc. -> (none); MF Diodes Inc. -> (none); MP AP2112K-3.3TRG1 -> (none); MPN (none) -> AP2112K-3.3TRG1; Manufacturer (none) -> Diodes Inc.; PARTREV 2-2 -> (none); Price None -> (none); SnapEDA_Link https://www.snapeda.com/parts/AP2112K-3.3TRG1/Diodes+Inc./v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 -> (none)

Commit message: hardware: Layout improvement
Parts:
- D_RPP_GATE1, Q_RPP1, R_RPP1: now not fitted
- L_BUCK1: footprint Inductor_SMD:L_Bourns-SRN6028 -> SparrowHawk:L_Sunlord_SWPA6028S; MPN (none) -> SWPA6028S6R8MT; Manufacturer (none) -> Sunlord; Note SRN6028 zostaje - zapas na nasycenie przy zwarciu +5V. SRN5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 -> Bourns SRN6028 jest wycofany z produkcji (EOL). Land patter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; Spec 6.8uH, Isat>=2.5A, Irms>=1.5A, DCR<=80mOhm -> 6,8 µH ±20 %, Isat ≥ 2,6 A, Irms ≥ 2,4 A, DCR ≤ 61 mΩ
- L_VID1: Spec (none) -> 4,7 µH ±20 %, Isat ≥ 1,1 A, DCR ≤ 163 mΩ, obudowa 3×3×1,5 mm

Commit message: hardware: finished board with sparrowhawk silkscreen
Parts:
- J_BAT1: now left out of the parts list
Connections:
- net VBAT_IN: no longer names the net of Q_RPP1.3 (D)
- no-connect marks 1 -> 2
Changed lines of the file:
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@@
 		)
 	)
-	(wire
-		(pts
-			(xy 100.33 76.2) (xy 106.68 76.2)
-		)
-		(stroke
-			(width 0)
-			(type default)
-		)
+	(no_connect
+		(at 100.33 76.2)
 	)
 	(wire
@@
 			(width 0)
 			(type default)
-		)
-	)
-	(label "VBAT_IN"
-		(at 106.68 76.2 0)
-		(effects
-			(font
-				(size 1.27 1.27)
-			)
-			(justify left bottom)
 		)
 	)
@@
 		(body_style 1)
 		(exclude_from_sim no)
-		(in_bom yes)
+		(in_bom no)
 		(on_board yes)
 		(in_pos_files yes)
