File: hardware/Sparrow-III/Interfaces&IO.kicad_sch (KiCad schematic)
At the start: 21 parts

Commit message: WIP: uncommitted changes, moved to the cloud
Snapshot of the working tree the Claude desktop app took to continue
this session in the cloud. It was never committed on the desktop; fold
it into your next commit (git commit --amend) or unstage it
(git reset --mixed HEAD~1) before committing for real.
Parts:
- C_CURR_F1: LCSC (none) -> C172740; MPN (none) -> C0402C105K4PACTU; Manufacturer (none) -> KEMET; Manufacturer_Name (none) -> KEMET; Manufacturer_Part_Number (none) -> C0402C105K4PACTU; Note (none) -> 1uF +/-10%, X5R, 16V, 0402. Selected in-stock procurement p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
- D_USB_VBUS1: LCSC (none) -> C110921
- J_ESC1: LCSC (none) -> C160394; Note PINOUT DO USTALENIA po wyborze 4in1 ESC - przepisac 1:1 z i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 -> FC pinout fixed; custom harness must map selected ESC signa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
- J_GPS1: LCSC (none) -> C160392; MPN BM06B-SRSS-TB (LF)(SN) -> BM06B-SRSS-TB(LF)(SN); Manufacturer_Part_Number (none) -> BM06B-SRSS-TB(LF)(SN)
- J_USB1: LCSC (none) -> C3197885
- R_CC1, R_CC2: LCSC (none) -> C105872; MPN (none) -> RC0402FR-075K1L; Manufacturer (none) -> YAGEO; Manufacturer_Name (none) -> YAGEO; Manufacturer_Part_Number (none) -> RC0402FR-075K1L; Note (none) -> 0402 thick-film, +/-1%, 0.063W. Voltage/power derating appl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
- R_CURR_F1: LCSC (none) -> C106235; MPN (none) -> RC0402FR-071KL; Manufacturer (none) -> YAGEO; Manufacturer_Name (none) -> YAGEO; Manufacturer_Part_Number (none) -> RC0402FR-071KL; Note (none) -> 0402 thick-film, +/-1%, 0.063W. Voltage/power derating appl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
- R_USB_SH1: LCSC (none) -> C242160; MPN (none) -> ERJ-2GE0R00X; Manufacturer (none) -> Panasonic; Manufacturer_Name (none) -> Panasonic; Manufacturer_Part_Number (none) -> ERJ-2GE0R00X; Note ekran USB-C wprost do GND (plytka ma jedna mase). Wczesniej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 -> 0ohm jumper, 0402; direct USB shield-to-GND connection.
- U_ESD1: LCSC (none) -> C7519
Changed lines of the file:
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@@
 			)
 		)
-		(property "Datasheet" ""
+		(property "Datasheet" "https://yageogroup.com/component-documentation/download/specsheet/RC0402FR-075K1L"
 			(at 113.03 91.44 0)
 			(hide yes)
@@
 			)
 		)
-		(property "Manufacturer_Name" ""
+		(property "Manufacturer_Name" "YAGEO"
 			(at 113.03 91.44 0)
 			(hide yes)
@@
 			)
 		)
-		(property "Manufacturer_Part_Number" ""
+		(property "Manufacturer_Part_Number" "RC0402FR-075K1L"
 			(at 113.03 91.44 0)
 			(hide yes)
@@
 			)
 		)
-	)
+ (property "MPN" "RC0402FR-075K1L" (at 113.03 91.44 0) (hide yes) (effects (font (size 1.27 1.27))))
+ (property "Manufacturer" "YAGEO" (at 113.03 91.44 0) (hide yes) (effects (font (size 1.27 1.27))))
+ (property "Note" "0402 thick-film, +/-1%, 0.063W. Voltage/power derating applies." (at 113.03 91.44 0) (hide yes) (effects (font (size 1.27 1.27))))
+ (property "LCSC" "C105872" (at 113.03 91.44 0) (hide yes) (effects (font (size 1.27 1.27)))))
 	(symbol
 		(lib_id "power:GND")
@@
 			)
 		)
-		(property "MPN" "BM06B-SRSS-TB (LF)(SN)"
+		(property "MPN" "BM06B-SRSS-TB(LF)(SN)"
 			(at 344.17 153.67 0)
 			(hide yes)
@@
 			)
 		)
-		(property "Manufacturer_Part_Number" ""
+		(property "Manufacturer_Part_Number" "BM06B-SRSS-TB(LF)(SN)"
 			(at 344.17 153.67 0)
 			(hide yes)
@@
 			)
 		)
-	)
+ (property "LCSC" "C160392" (at 344.17 153.67 0) (hide yes) (effects (font (size 1.27 1.27)))))
 	(symbol
 		(lib_id "Device:C")
@@
 			)
 		)
-	)
+ (property "LCSC" "C110921" (at 153.67 63.5 180) (hide yes) (effects (font (size 1.27 1.27)))))
 	(symbol
 		(lib_id "power:+5V")
@@
 			)
 		)
-		(property "Note" "PINOUT DO USTALENIA po wyborze 4in1 ESC - przepisac 1:1 z instrukcji"
+		(property "Note" "FC pinout fixed; custom harness must map selected ESC signals. Do not assume1:1 cable. With J_BAT input, omit ESC VBAT conductor; retain common GND."
 			(at 347.98 100.33 0)
 			(hide yes)
@@
 			)
 		)
-	)
+ (property "LCSC" "C160394" (at 347.98 100.33 0) (hide yes) (effects (font (size 1.27 1.27)))))
 	(symbol
 		(lib_id "power:GND")
@@
 			)
 		)
-		(property "Datasheet" ""
+		(property "Datasheet" "https://yageogroup.com/component-documentation/download/specsheet/RC0402FR-075K1L"
 			(at 124.46 91.44 0)
 			(hide yes)
@@
 			)
 		)
-		(property "Manufacturer_Name" ""
+		(property "Manufacturer_Name" "YAGEO"
 			(at 124.46 91.44 0)
 			(hide yes)
@@
 			)
 		)
-		(property "Manufacturer_Part_Number" ""
+		(property "Manufacturer_Part_Number" "RC0402FR-075K1L"
 			(at 124.46 91.44 0)
 			(hide yes)
@@
 			)
 		)
-	)
+ (property "MPN" "RC0402FR-075K1L" (at 124.46 91.44 0) (hide yes) (effects (font (size 1.27 1.27))))
+ (property "Manufacturer" "YAGEO" (at 124.46 91.44 0) (hide yes) (effects (font (size 1.27 1.27))))
+ (property "Note" "0402 thick-film, +/-1%, 0.063W. Voltage/power derating applies." (at 124.46 91.44 0) (hide yes) (effects (font (size 1.27 1.27))))
+ (property "LCSC" "C105872" (at 124.46 91.44 0) (hide yes) (effects (font (size 1.27 1.27)))))
 	(symbol
 		(lib_id "power:GND")
@@
 			)
 		)
-		(property "Datasheet" ""
+		(property "Datasheet" "https://search.kemet.com/download/specsheet/C0402C105K4PACTU"
 			(at 261.62 97.79 0)
 			(hide yes)
@@
 			)
 		)
-		(property "Manufacturer_Name" ""
+		(property "Manufacturer_Name" "KEMET"
 			(at 261.62 97.79 0)
 			(hide yes)
@@
 			)
 		)
-		(property "Manufacturer_Part_Number" ""
+		(property "Manufacturer_Part_Number" "C0402C105K4PACTU"
 			(at 261.62 97.79 0)
 			(hide yes)
@@
 			)
 		)
-	)
+ (property "MPN" "C0402C105K4PACTU" (at 261.62 97.79 0) (hide yes) (effects (font (size 1.27 1.27))))
+ (property "Manufacturer" "KEMET" (at 261.62 97.79 0) (hide yes) (effects (font (size 1.27 1.27))))
+ (property "Note" "1uF +/-10%, X5R, 16V, 0402. Selected in-stock procurement part; qualify ADC settling and VDDA noise on prototype." (at 261.62 97.79 0) (hide yes) (effects (font (size 1.27 1.27))))
+ (property "LCSC" "C172740" (at 261.62 97.79 0) (hide yes) (effects (font (size 1.27 1.27)))))
 	(symbol
 		(lib_id "Device:R")
@@
 			)
 		)
-		(property "Datasheet" ""
+		(property "Datasheet" "https://industrial.panasonic.com/ww/products/pt/chip-resistors/models/ERJ2GE0R00X"
 			(at 76.2 99.06 0)
 			(hide yes)
@@
 			)
 		)
-		(property "Note" "ekran USB-C wprost do GND (plytka ma jedna mase). Wczesniej 1M || 10nF"
+		(property "Note" "0ohm jumper, 0402; direct USB shield-to-GND connection."
 			(at 76.2 99.06 0)
 			(hide yes)
@@
 			)
 		)
-		(property "Manufacturer_Name" ""
+		(property "Manufacturer_Name" "Panasonic"
 			(at 76.2 99.06 0)
 			(hide yes)
@@
 			)
 		)
-		(property "Manufacturer_Part_Number" ""
+		(property "Manufacturer_Part_Number" "ERJ-2GE0R00X"
 			(at 76.2 99.06 0)
 			(hide yes)
@@
 			)
 		)
-	)
+ (property "MPN" "ERJ-2GE0R00X" (at 76.2 99.06 0) (hide yes) (effects (font (size 1.27 1.27))))
+ (property "Manufacturer" "Panasonic" (at 76.2 99.06 0) (hide yes) (effects (font (size 1.27 1.27))))
+ (property "LCSC" "C242160" (at 76.2 99.06 0) (hide yes) (effects (font (size 1.27 1.27)))))
 	(symbol
 		(lib_id "BM04B-SRSS-TB_LF__SN_:BM04B-SRSS-TB_LF__SN_")
@@
 			)
 		)
- (property "Mounting" "Horizontal top mount; body inside PCB; entry from right edge" (at 83.82 71.12 0) (hide yes) (effects (font (size 1.27 1.27)))))
+ (property "Mounting" "Horizontal top mount; body inside PCB; entry from right edge" (at 83.82 71.12 0) (hide yes) (effects (font (size 1.27 1.27))))
+ (property "LCSC" "C3197885" (at 83.82 71.12 0) (hide yes) (effects (font (size 1.27 1.27)))))
 	(symbol
 		(lib_id "power:GND")
@@
 			)
 		)
-		(property "Datasheet" ""
+		(property "Datasheet" "https://yageogroup.com/component-documentation/download/specsheet/RC0402FR-071KL"
 			(at 275.59 93.98 0)
 			(hide yes)
@@
 			)
 		)
-		(property "Manufacturer_Name" ""
+		(property "Manufacturer_Name" "YAGEO"
 			(at 275.59 93.98 90)
 			(hide yes)
@@
 			)
 		)
-		(property "Manufacturer_Part_Number" ""
+		(property "Manufacturer_Part_Number" "RC0402FR-071KL"
 			(at 275.59 93.98 90)
 			(hide yes)
@@
 			)
 		)
-	)
+ (property "MPN" "RC0402FR-071KL" (at 275.59 93.98 90) (hide yes) (effects (font (size 1.27 1.27))))
+ (property "Manufacturer" "YAGEO" (at 275.59 93.98 90) (hide yes) (effects (font (size 1.27 1.27))))
+ (property "Note" "0402 thick-film, +/-1%, 0.063W. Voltage/power derating applies." (at 275.59 93.98 90) (hide yes) (effects (font (size 1.27 1.27))))
+ (property "LCSC" "C106235" (at 275.59 93.98 90) (hide yes) (effects (font (size 1.27 1.27)))))
 	(symbol
 		(lib_id "Power_Protection:USBLC6-2SC6")
@@
 			)
 		)
-	)
+ (property "LCSC" "C7519" (at 153.67 88.9 0) (hide yes) (effects (font (size 1.27 1.27)))))
 	(symbol
 		(lib_id "Device:Buzzer")
