File: hardware/Sparrow-III/Interfaces&IO.kicad_sch (KiCad schematic)
At the start: 21 parts

Commit message: hardware: Sparrow III interfaces and IO sheet rework
Parts:
- C_CURR_F1: LCSC (none) -> C172740; MPN (none) -> C0402C105K4PACTU; Manufacturer (none) -> KEMET; Manufacturer_Name (none) -> KEMET; Manufacturer_Part_Number (none) -> C0402C105K4PACTU; Note (none) -> 1uF +/-10%, X5R, 16V, 0402. Selected in-stock procurement p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
- D_USB_VBUS1: LCSC (none) -> C110921
- J_ESC1: LCSC (none) -> C160394; Note PINOUT DO USTALENIA po wyborze 4in1 ESC - przepisac 1:1 z i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 -> FC pinout fixed; custom harness must map selected ESC signa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
- J_GPS1: LCSC (none) -> C160392; MPN BM06B-SRSS-TB (LF)(SN) -> BM06B-SRSS-TB(LF)(SN); Manufacturer_Part_Number (none) -> BM06B-SRSS-TB(LF)(SN)
- J_USB1: LCSC (none) -> C3197885
- R_CC1, R_CC2: LCSC (none) -> C105872; MPN (none) -> RC0402FR-075K1L; Manufacturer (none) -> YAGEO; Manufacturer_Name (none) -> YAGEO; Manufacturer_Part_Number (none) -> RC0402FR-075K1L; Note (none) -> 0402 thick-film, +/-1%, 0.063W. Voltage/power derating appl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
- R_CURR_F1: LCSC (none) -> C106235; MPN (none) -> RC0402FR-071KL; Manufacturer (none) -> YAGEO; Manufacturer_Name (none) -> YAGEO; Manufacturer_Part_Number (none) -> RC0402FR-071KL; Note (none) -> 0402 thick-film, +/-1%, 0.063W. Voltage/power derating appl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
- R_USB_SH1: LCSC (none) -> C242160; MPN (none) -> ERJ-2GE0R00X; Manufacturer (none) -> Panasonic; Manufacturer_Name (none) -> Panasonic; Manufacturer_Part_Number (none) -> ERJ-2GE0R00X; Note ekran USB-C wprost do GND (plytka ma jedna mase). Wczesniej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 -> 0ohm jumper, 0402; direct USB shield-to-GND connection.
- U_ESD1: LCSC (none) -> C7519
