File: hardware/Sparrow-III/MCU.kicad_sch (KiCad schematic)
At the start: 27 parts

Commit message: WIP: uncommitted changes, moved to the cloud
Snapshot of the working tree the Claude desktop app took to continue
this session in the cloud. It was never committed on the desktop; fold
it into your next commit (git commit --amend) or unstage it
(git reset --mixed HEAD~1) before committing for real.
Parts:
- C_HSE1, C_HSE2: LCSC (none) -> C161527; MPN (none) -> GRM1555C1H120GA01D; Manufacturer (none) -> Murata; Manufacturer_Name (none) -> Murata; Manufacturer_Part_Number (none) -> GRM1555C1H120GA01D; Note (none) -> 12pF +/-2%, C0G/NP0, 50V, 0402. Prototype starting loads; e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
- C_NRST1, C_VDD1, C_VDD2, C_VDD3, C_VDD4, C_VDDA_HF1: LCSC (none) -> C77020; MPN (none) -> GRM155R71H104KE14D; Manufacturer (none) -> Murata; Manufacturer_Name (none) -> Murata; Manufacturer_Part_Number (none) -> GRM155R71H104KE14D; Note (none) -> 100nF +/-10%, X7R, 50V, 0402. Manufacturer reference sheet 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; Voltage 16V -> 50V
- C_VCAP1: LCSC (none) -> C87998; MPN (none) -> CL21B475KPFNNNE; Manufacturer (none) -> Samsung Electro-Mechanics; Manufacturer_Name TDK -> Samsung Electro-Mechanics; Manufacturer_Part_Number C2012X7R1A475K125AC -> CL21B475KPFNNNE; Note (none) -> 4.7uF +/-10%, X7R, 10V, 0805; VCAP. Branch ESR set by R_VCA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
- C_VDDA1: LCSC (none) -> C172740; MPN (none) -> C0402C105K4PACTU; Manufacturer (none) -> KEMET; Manufacturer_Name (none) -> KEMET; Manufacturer_Part_Number (none) -> C0402C105K4PACTU; Note (none) -> 1uF +/-10%, X5R, 16V, 0402. Selected in-stock procurement p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
- C_VDD_BULK1: LCSC (none) -> C77045; MPN (none) -> GRM188R61C475KE11D; Manufacturer (none) -> Murata; Manufacturer_Name (none) -> Murata; Manufacturer_Part_Number (none) -> GRM188R61C475KE11D; Note (none) -> 4.7uF +/-10%, X5R, 16V, 0603; supplementary MCU bulk.
- FB_VDDA1: LCSC (none) -> C356953; MPN (none) -> HCB1005KF-101T10; Manufacturer (none) -> TAI-TECH; Manufacturer_Name (none) -> TAI-TECH; Manufacturer_Part_Number (none) -> HCB1005KF-101T10; Note (none) -> 100ohm +/-25% at 100MHz, 0402, 1A, DCR 0.2ohm; VDDA filter.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
- LED_PWR1: LCSC (none) -> C125094; MPN (none) -> LTST-C190KGKT; Manufacturer (none) -> Lite-On; Manufacturer_Name (none) -> Lite-On; Manufacturer_Part_Number (none) -> LTST-C190KGKT; Note (none) -> 0603 green indicator; KiCad pad1=cathode, pad2=anode. Verif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
- LED_STAT1: LCSC (none) -> C125096; MPN (none) -> LTST-C190TBKT; Manufacturer (none) -> Lite-On; Manufacturer_Name (none) -> Lite-On; Manufacturer_Part_Number (none) -> LTST-C190TBKT; Note (none) -> 0603 blue indicator; KiCad pad1=cathode, pad2=anode. Verify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
- LED_STAT2: LCSC (none) -> C94869; MPN (none) -> LTST-C190KRKT; Manufacturer (none) -> Lite-On; Manufacturer_Name (none) -> Lite-On; Manufacturer_Part_Number (none) -> LTST-C190KRKT; Note (none) -> 0603 red indicator; KiCad pad1=cathode, pad2=anode. Verify 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
- R_BOOT0: LCSC (none) -> C60490; MPN (none) -> RC0402FR-0710KL; Manufacturer (none) -> YAGEO; Manufacturer_Name (none) -> YAGEO; Manufacturer_Part_Number (none) -> RC0402FR-0710KL; Note (none) -> 0402 thick-film, +/-1%, 0.063W. Voltage/power derating appl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
- R_HSE2: LCSC (none) -> C242160; MPN (none) -> ERJ-2GE0R00X; Manufacturer (none) -> Panasonic; Manufacturer_Name (none) -> Panasonic; Manufacturer_Part_Number (none) -> ERJ-2GE0R00X; Note (none) -> 0ohm jumper, 0402; series HSE tuning position, initially po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
- R_I2C_SCL1, R_I2C_SDA1: LCSC (none) -> C105871; MPN (none) -> RC0402FR-074K7L; Manufacturer (none) -> YAGEO; Manufacturer_Name (none) -> YAGEO; Manufacturer_Part_Number (none) -> RC0402FR-074K7L; Note (none) -> 0402 thick-film, +/-1%, 0.063W. Voltage/power derating appl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
- R_LED1, R_LED2, R_LED3: LCSC (none) -> C106235; MPN (none) -> RC0402FR-071KL; Manufacturer (none) -> YAGEO; Manufacturer_Name (none) -> YAGEO; Manufacturer_Part_Number (none) -> RC0402FR-071KL; Note (none) -> 0402 thick-film, +/-1%, 0.063W. Voltage/power derating appl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
- R_VCAP_ESR1: LCSC (none) -> C45879; MPN (none) -> 0603WAF150LT5E; Manufacturer (none) -> UNI-ROYAL; Manufacturer_Name Panasonic -> UNI-ROYAL; Manufacturer_Part_Number ERJ3RSFR15V -> 0603WAF150LT5E; Note (none) -> 0.15ohm +/-1%, 0.1W, 0603, TCR 800ppm/K; VCAP series ESR, b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
- U_MCU1: LCSC (none) -> C118207
- Y_HSE1: value 8MHz CL=10pF ESR<150R -> 8MHz; LCSC (none) -> C2682775; MPN (none) -> X32258MOB4SI; Manufacturer (none) -> YXC; Manufacturer_Name (none) -> YXC; Manufacturer_Part_Number (none) -> X32258MOB4SI; Note (none) -> 8MHz, CL 12pF, ESR max 180ohm, +/-10ppm/+/-20ppm, 3225-4P, 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; Spec 8 MHz, CL = 10 pF, ESR ≤ 150 Ω, obudowa 3225 4-pad (C_HSE1/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 -> 8MHz; CL12pF; ESR150ohm custom R150 option; C0 max2pF; driv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
