File: hardware/Sparrow-III/Power.kicad_sch (KiCad schematic)
At the start: 35 parts

Commit message: WIP: uncommitted changes, moved to the cloud
Snapshot of the working tree the Claude desktop app took to continue
this session in the cloud. It was never committed on the desktop; fold
it into your next commit (git commit --amend) or unstage it
(git reset --mixed HEAD~1) before committing for real.
Parts:
- C_3V3_BULK1, C_5V_BULK1: LCSC (none) -> C92487; MPN (none) -> CL10A106MO8NQNC; Manufacturer (none) -> Samsung Electro-Mechanics; Manufacturer_Name (none) -> Samsung Electro-Mechanics; Manufacturer_Part_Number (none) -> CL10A106MO8NQNC; Note (none) -> 10uF +/-20%, X5R, 16V, 0603; supplemental bulk. Replaces TD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
- C_B1, C_B5: LCSC (none) -> C92059
- C_BUCK_BOOT1: LCSC (none) -> C77020; MPN (none) -> GRM155R71H104KE14D; Manufacturer (none) -> Murata; Manufacturer_Name (none) -> Murata; Manufacturer_Part_Number (none) -> GRM155R71H104KE14D; Note (none) -> 100nF +/-10%, X7R, 50V, 0402. Manufacturer reference sheet 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
- C_BUCK_IN1: LCSC (none) -> C342614; MPN (none) -> C3225X7S2A475KT000N; Manufacturer (none) -> TDK; Manufacturer_Name (none) -> TDK; Manufacturer_Part_Number (none) -> C3225X7S2A475KT000N; Note 100V wg TI SNVSA81B (2x Vin); przy 25V bias ok. 2uF efektyw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 -> 4.7uF +/-10%, X7S, 100V, 1210; buck input. Same TDK C3225 X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
- C_BUCK_IN2: LCSC (none) -> C342614; MPN (none) -> C3225X7S2A475KT000N; Manufacturer (none) -> TDK; Manufacturer_Name (none) -> TDK; Manufacturer_Part_Number (none) -> C3225X7S2A475KT000N; Note (none) -> 4.7uF +/-10%, X7S, 100V, 1210; buck input. Same TDK C3225 X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
- C_BUCK_IN3: LCSC (none) -> C77058; MPN (none) -> GRM188R72A104KA35D; Manufacturer (none) -> Murata; Manufacturer_Name (none) -> Murata; Manufacturer_Part_Number (none) -> GRM188R72A104KA35D; Note (none) -> 100nF +/-10%, X7R, 100V, 0603; local high-frequency VIN byp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
- C_BUCK_OUT1: value 47uF -> 100uF; LCSC (none) -> C394395; MPN (none) -> EMK325ABJ107MM-T; Manufacturer (none) -> Taiyo Yuden; Manufacturer_Name (none) -> Taiyo Yuden; Manufacturer_Part_Number (none) -> EMK325ABJ107MM-T; Note (none) -> 100uF +/-20%, X5R, 16V, 1210; buck output. 16V rating keeps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
- C_BUCK_SS1: LCSC (none) -> C77010; MPN (none) -> GRM155R71C223KA01D; Manufacturer (none) -> Murata; Manufacturer_Name (none) -> Murata; Manufacturer_Part_Number (none) -> GRM155R71C223KA01D; Note (none) -> 22nF +/-10%, X7R, 16V, 0402; soft-start timing.
- C_LDO_IN1, C_LDO_OUT1: value 1uF -> 2.2uF; footprint Capacitor_SMD:C_0402_1005Metric -> Capacitor_SMD:C_0603_1608Metric; LCSC (none) -> C415535; MPN (none) -> GRM188Z71E225KE43D; Manufacturer (none) -> Murata; Manufacturer_Name (none) -> Murata; Manufacturer_Part_Number (none) -> GRM188Z71E225KE43D; Note (none) -> 2.2uF +/-10%, X7R, 25V, 0603; LDO in/out. TLV755P SBVS320D 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; Voltage 16V -> 25V
- C_VBAT_ADC1: LCSC (none) -> C77020; MPN (none) -> GRM155R71H104KE14D; Manufacturer (none) -> Murata; Manufacturer_Name (none) -> Murata; Manufacturer_Part_Number (none) -> GRM155R71H104KE14D; Note (none) -> 100nF +/-10%, X7R, 50V, 0402. Manufacturer reference sheet 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; Voltage 16V -> 50V
- D_BUCK1: LCSC (none) -> C283521
- D_TVS1: value SMAJ28A -> SMAJ26A; LCSC (none) -> C148225; MPN SMAJ28A -> SMAJ26A; Manufacturer_Name (none) -> Littelfuse; Manufacturer_Part_Number (none) -> SMAJ26A; Note Vwm 28V, Vc 45.4V @8.8A. Uwaga: LMR14030 ma abs.max VIN = 4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 -> 4S-6S conventional LiPo only, max steady input 25.2V. Vwm=2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
- L_BUCK1: footprint SparrowHawk:L_Sunlord_SWPA6028S -> SparrowHawk:L_Vishay_IHLP-2525CZ-01; LCSC (none) -> C506575; MPN SWPA6028S6R8MT -> IHLP2525CZER6R8M01; Manufacturer Sunlord -> Vishay; Manufacturer_Name (none) -> Vishay; Manufacturer_Part_Number (none) -> IHLP2525CZER6R8M01; Note Bourns SRN6028 jest wycofany z produkcji (EOL). Land patter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 -> 6.8uH +/-20%; Isat typ8A at 20% L drop/25C; heat rating typ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
- R_BUCK_FB1, R_VBAT_D1: LCSC (none) -> C60491; MPN (none) -> RC0402FR-07100KL; Manufacturer (none) -> YAGEO; Manufacturer_Name (none) -> YAGEO; Manufacturer_Part_Number (none) -> RC0402FR-07100KL; Note (none) -> 0402 thick-film, +/-1%, 0.063W. Voltage/power derating appl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
- R_BUCK_FB2: LCSC (none) -> C185458; MPN (none) -> RC0402FR-0717K8L; Manufacturer (none) -> YAGEO; Manufacturer_Name (none) -> YAGEO; Manufacturer_Part_Number (none) -> RC0402FR-0717K8L; Note (none) -> 0402 thick-film, +/-1%, 0.063W. Voltage/power derating appl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
- R_BUCK_RT1: LCSC (none) -> C2076619; MPN (none) -> CR0402-FX-4992GLF; Manufacturer (none) -> Bourns; Manufacturer_Name (none) -> Bourns; Manufacturer_Part_Number (none) -> CR0402-FX-4992GLF; Note (none) -> 49.9k +/-1%, 0402, 0.063W; selected in-stock part for buck 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
- R_VBAT_D2: LCSC (none) -> C60490; MPN (none) -> RC0402FR-0710KL; Manufacturer (none) -> YAGEO; Manufacturer_Name (none) -> YAGEO; Manufacturer_Part_Number (none) -> RC0402FR-0710KL; Note (none) -> 0402 thick-film, +/-1%, 0.063W. Voltage/power derating appl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
- U_BUCK1: LCSC (none) -> C182078
- U_LDO1: value AP2112K-3.3TRG1 -> TLV75533PDYDR; footprint Package_TO_SOT_SMD:SOT-23-5 -> SparrowHawk:SOT-23-5_ThermalPad_TI_DYD0005A; symbol AP2112K-3.3TRG1:AP2112K-3.3TRG1 -> TLV75533PDYD:TLV75533PDYD; LCSC (none) -> C28642215; MPN AP2112K-3.3TRG1 -> TLV75533PDYDR; Manufacturer Diodes Inc. -> Texas Instruments; Manufacturer_Name (none) -> Texas Instruments; Manufacturer_Part_Number (none) -> TLV75533PDYDR; Note (none) -> 300mA board design budget; VIN<=5.5V. Thermal pad6 to GND w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; Package SOT-753 Diodes Inc. -> TI DYD0005A SOT-23-5 with thermal pad
Connections:
- net GND: now also U_LDO1.6 (EP); no longer U_LDO1.4 (SH)
- no-connect marks 2 -> 3
