File: hardware/Sparrow-III/Sensors.kicad_sch (KiCad schematic)
At the start: 19 parts

Commit message: hardware: Sparrow III sensors sheet rework
Parts:
- C_BARO1, C_BARO2, C_FLASH1, C_IMU_VDD2, C_IMU_VIO1: LCSC (none) -> C77020; MPN (none) -> GRM155R71H104KE14D; Manufacturer (none) -> Murata; Manufacturer_Name (none) -> Murata; Manufacturer_Part_Number (none) -> GRM155R71H104KE14D; Note (none) -> 100nF +/-10%, X7R, 50V, 0402. Manufacturer reference sheet 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; Voltage 16V -> 50V
- C_IMU_VDD1: LCSC (none) -> C88944; MPN (none) -> GRM155R61C225KE11D; Manufacturer (none) -> Murata; Manufacturer_Name (none) -> Murata; Manufacturer_Part_Number (none) -> GRM155R61C225KE11D; Note (none) -> 2.2uF +/-10%, X5R, 16V, 0402; local IMU decoupling; nominal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
- C_IMU_VIO2: LCSC (none) -> C85735; MPN (none) -> GRM155R71C103KA01D; Manufacturer (none) -> Murata; Manufacturer_Name (none) -> Murata; Manufacturer_Part_Number (none) -> GRM155R71C103KA01D; Note (none) -> 10nF +/-10%, X7R, 16V, 0402; IMU VDDIO high-frequency decou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
- C_MAG_BULK1: value 10uF -> 22uF; LCSC (none) -> C98190; MPN (none) -> CL21A226MOQNNNE; Manufacturer (none) -> Samsung Electro-Mechanics; Manufacturer_Name (none) -> Samsung Electro-Mechanics; Manufacturer_Part_Number (none) -> CL21A226MOQNNNE; Note 10uF ceramic X5R/X7R, 0805. Verify effective capacitance at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 -> 22uF +/-20%, X5R, 16V, 0805; LIS2MDL local bulk.
- C_MAG_SET1: LCSC (none) -> C16772; MPN (none) -> CL05B224KO5NNNC; Manufacturer (none) -> Samsung Electro-Mechanics; Manufacturer_Name (none) -> Samsung Electro-Mechanics; Manufacturer_Part_Number (none) -> CL05B224KO5NNNC; Note 220nF ceramic X7R, ESR <=200mOhm per LIS2MDL application ci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 -> 220nF +/-10%, X7R, 16V, 0402; LIS2MDL C1 set/reset capacito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
- C_MAG_VDD1: LCSC (none) -> C77020; MPN (none) -> GRM155R71H104KE14D; Manufacturer (none) -> Murata; Manufacturer_Name (none) -> Murata; Manufacturer_Part_Number (none) -> GRM155R71H104KE14D; Note 100nF ceramic X7R; VDD pin 9 local decoupling -> 100nF +/-10%, X7R, 50V, 0402. Manufacturer reference sheet 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; Voltage 16V -> 50V
- C_MAG_VIO1: LCSC (none) -> C77020; MPN (none) -> GRM155R71H104KE14D; Manufacturer (none) -> Murata; Manufacturer_Name (none) -> Murata; Manufacturer_Part_Number (none) -> GRM155R71H104KE14D; Note 100nF ceramic X7R; VDDIO pin 10 local decoupling -> 100nF +/-10%, X7R, 50V, 0402. Manufacturer reference sheet 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; Voltage 16V -> 50V
- FB_IMU1: LCSC (none) -> C76884; MPN (none) -> BLM15AG601SN1D; Manufacturer (none) -> Murata; Manufacturer_Name (none) -> Murata; Manufacturer_Part_Number (none) -> BLM15AG601SN1D; Note (none) -> 600ohm +/-25% at100MHz, 0402, rated300mA, DCR max0.52ohm. L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
- R_FLASH_CS1, R_FLASH_HD1, R_FLASH_WP1: LCSC (none) -> C60490; MPN (none) -> RC0402FR-0710KL; Manufacturer (none) -> YAGEO; Manufacturer_Name (none) -> YAGEO; Manufacturer_Part_Number (none) -> RC0402FR-0710KL; Note (none) -> 0402 thick-film, +/-1%, 0.063W. Voltage/power derating appl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
- U_BARO1: value DPS310 -> DPS368; LCSC (none) -> C3232508; MPN DPS310 -> DPS368XTSA1; Manufacturer_Name (none) -> Infineon Technologies; Manufacturer_Part_Number (none) -> DPS368XTSA1; Note (none) -> Baro: DPS310XTSA1 discontinued at LCSC/JLC. DPS368 has the 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
- U_FLASH1: LCSC (none) -> C190862
- U_IMU1: LCSC (none) -> C1850418
- U_MAG1: LCSC (none) -> C919695
Other:
- note added: "Magnetometr"
- note removed: "Magnetometr — LIS2MDL / I2C1"
- note removed: "Sparrow III: LIS2MDL, I2C1 @ 0x1E. C1=220nF low ESR <=200mR. GPS: choose compass with address other than 0x1E, or leave GPS I2C unconnected. LGA requires controlled reflow / hot air; do not attempt iron-only assembly."
